File: KiCad/EEZ DIB DCP405plus.kicad_pcb (KiCad board)
At the start: 4 copper layers, 180 x 103.5 mm, 424 parts, among them IC1 ADS131A04IPBSR, IC10 TC77-5.0MCTTR, IC11 REF5025AIDR, IC12 MC79L05, IC13 MC78L05, IC14 PCAL9722HNMP, IC15 TPS7A2033PDBVR, IC16 LM5145RGYR, IC17 LTC2050HVCS8#PBF, IC18 TL072D, IC19 TL072D, IC2 ISO6762FDWR, IC20 SN74LVC1G3157DCKR, IC21 SN74LVC2G08DCTR, IC22 LM293D, IC23 OPA376AIDBVR, IC24 SN74LVC1G3157DCKR, IC25 SN74LVC1G3157DCKR, IC26 LM293D, IC27 MAX9141ESA, IC3 ISO6762FDWR, IC4 ISO6520DR, IC5 STM32H503CBT6, IC6 M24C32-DFDW6TP, IC7 DAC8552IDGKR, IC8 74AUP1G74DC,125, IC9 TPS54060DGQ, J1 572-0500, J2 572-0100, K1 FTR-C1GA012G-B05 or EE2-12NU-L, Q1 BSS84, Q10 MMBT5401, Q11 MMBT5401, Q12 BCP56-16.115, Q13 MMBT5551, Q14 IRFP250NPBF, Q15 BCP56-16.115, Q16 BC857C, Q17 IRFI9Z34GPBF, Q18 PSMN0R9-25YLC, Q19 PSMN0R9-25YLC, Q2 BSS84, Q20 MMBT5551, Q21 MMBT5551, Q22 MMBT5551, Q23 MMBT5401, Q24 2N7002, Q25 2N7002, Q26 2N7002, Q27 2N7002, Q28 MMBT5551, Q29 FMMT493TA, Q3 BSS84, Q30 BT139B-600E, Q31 PSMN013-60YL, Q4 BSC117N08NS5ATMA1, Q5 BSC039N06NSATMA1, Q6 2N7002, Q7 MMBT5401, Q8 DMP6023LFG-7, Q9 MMBT5551, X1 Edge connector, X2 N.C., X3 B4P-VH (LF)(SN), X4 TBP03R1-350-03BE, X5 ZL263-20DG, Y1 ECS-163.84-10-33-JGN-TR, Y2 ABM8-25.000MHZ-D2X-T

Commit message: X3 type changed
Parts:
- X3: value B4P-VH (LF)(SN) -> B4PS-VH (LF)(SN); footprint PCM_EEZ_connectors:B4P-VH_LF_SN -> PCM_EEZ_connectors:B4PS-VH
- moved ZD2 16.0 mm to (218.7, 137.9), turned to -90 degrees
- moved X3 7.82 mm to (222.7, 135.0), turned to 90 degrees
- moved R34 6.80 mm to (218.8, 130.4), turned to 90 degrees
- moved FM4 2.00 mm to (220.0, 142.5)
- moved C61 0.70 mm to (228.8, 125.5)
- moved C63 0.44 mm to (226.0, 123.0)
- moved C65 0.44 mm to (231.5, 123.0)
Routing:
- net /Power pre-regulator/DC+: track 39.5 -> 27.0 mm
- net /Power pre-regulator/DC-: track 55.2 -> 61.7 mm
- net DC_OUT: track 182.6 -> 181.4 mm
Other:
- board text added: "EEZ DCP405+ (01/2026 ${project_version})"
- board text removed: "EEZ DCP405+ (12/2025 ${project_version})"

Commit message: DIB connector update
Parts:
- J1: footprint PCM_EEZ_connectors:572-0X00 -> PCM_EEZ_connectors:572-0500
- J2: footprint PCM_EEZ_connectors:572-0X00 -> PCM_EEZ_connectors:572-0100
- Q18, Q19: value PSMN0R9-25YLC -> IAUZ40N06S5N050ATMA1; footprint PCM_EEZ_SMD:SOT669 -> PCM_EEZ_SMD:TDSON-8
- X1: value Edge connector -> 10018783-10101TLF
- moved Q19 0.59 mm to (102.3, 57.2), turned to 180 degrees
- moved Q18 0.57 mm to (102.3, 63.1), turned to 180 degrees
- renumbered R94 to R93, R95 to R94, R93 to R95, R97 to R96, R96 to R97
Connections:
- X1 pad A1: unconnected-(X1-+12V-PadA1) -> PE
- X1 pad A8: PE -> unconnected-(X1-~{SHUTDOWN}-PadA8)
Routing:
- net DIB_3V3: track 25.0 -> 22.2 mm
- net PE: vias 4 -> 3
- net DIB_GND: vias 33 -> 32
