File: KiCad/EEZ DIB DCP405plus.kicad_pcb (KiCad board)
At the start: 4 copper layers, 180 x 103.5 mm, 430 parts, among them IC1 ADS131A04IPBSR, IC10 TC77-5.0MCTTR, IC11 REF5025AIDR, IC12 MC79L05, IC13 MC78L05, IC14 PCAL9722HNMP, IC15 TPS7A2033PDBVR, IC16 LM5145RGYR, IC17 LTC2050HVCS8#PBF, IC18 TL072D, IC19 TL072D, IC2 ISO6762FDWR, IC20 SN74LVC1G3157DCKR, IC21 SN74LVC2G08DCTR, IC22 LM293D, IC23 OPA376AIDBVR, IC24 SN74LVC1G3157DCKR, IC25 SN74LVC1G3157DCKR, IC26 LM293D, IC27 MAX9141ESA, IC3 ISO6762FDWR, IC4 ISO6520DR, IC5 STM32H503CBT6, IC6 M24C32-DFDW6TP, IC7 DAC8552IDGKR, IC8 74AUP1G74DC,125, IC9 TPS54060DGQ, J1 572-0500, J2 572-0100, K1 FTR-C1GA012G-B05 or EE2-12NU-L, Q1 BSS84, Q10 MMBT5401, Q11 MMBT5401, Q12 BCP56-16.115, Q13 MMBT5551, Q14 IRFP250NPBF, Q15 BCP56-16.115, Q16 BC857C, Q17 IRFI9Z34GPBF, Q18 PSMN0R9-25YLC, Q19 PSMN0R9-25YLC, Q2 BSS84, Q20 MMBT5551, Q21 MMBT5551, Q22 MMBT5551, Q23 MMBT5401, Q24 2N7002, Q25 2N7002, Q26 2N7002, Q27 2N7002, Q28 MMBT5551, Q29 FMMT493TA, Q3 BSS84, Q30 BT139B-600E, Q31 PSMN013-60YL, Q4 BSC117N08NS5ATMA1, Q5 BSC039N06NSATMA1, Q6 2N7002, Q7 MMBT5401, Q8 SQJ457EP-T1_BE3, Q9 MMBT5551, X1 PCB Edge connector, X2 N.C., X3 B4PS-VH (LF)(SN), X4 TBP03R1-350-03BE, X5 ZL263-20DG, Y1 ECS-163.84-10-33-JGN-TR, Y2 ABM8-25.000MHZ-D2X-T

Commit message: #4
Parts:
- added D24: BAS316, PCM_EEZ_SMD:SOD-323_1P8X1P35_ONS-M, F.Cu at (128.0, 139.0)
Connections:
- X1 pad A8: unconnected-(X1-~{SHUTDOWN}-PadA8) -> /DIB isolators, EEPROM, ADC, MCU/~{DIB_SHUTDOWN}
Routing:
- net /DIB isolators, EEPROM, ADC, MCU/~{DIB_SHUTDOWN}: track 0.00 -> 11.2 mm, vias 0 -> 1
- net GND: vias 119 -> 121

Commit message: #5
Parts:
- removed Q1, Q2: BSS84, PCM_EEZ_SMD:SOT103P240X110-3N
- removed R147, R148: 47K, PCM_EEZ_passives:R_0805_2012Metric
- R21: value 750R -> 1K8
- R22: value 6K2 -> 330R
Connections:
- LED1 pad GREEN: Net-(LED1-AG) -> /DAC, OE, Vref, IOEXP, Temp/~{OE_LED_GREEN}
- LED1 pad RED: Net-(LED1-AR) -> /DAC, OE, Vref, IOEXP, Temp/~{OE_LED_RED}
Routing:
- net Net-(LED1-AR): track 65.1 -> 0.00 mm, vias 2 -> 0
- net Net-(LED1-AG): track 56.4 -> 0.00 mm, vias 2 -> 0
- net /DAC, OE, Vref, IOEXP, Temp/~{OE_LED_RED}: track 58.6 -> 106.0 mm
- net /DAC, OE, Vref, IOEXP, Temp/~{OE_LED_GREEN}: track 56.4 -> 99.6 mm
- net +VLED: track 184.0 -> 177.9 mm, vias 4 -> 2
