File: KiCad/Bias_power.kicad_sch (KiCad schematic)
At the start: 42 parts, among them IC12 MC79L05, IC13 MC78L05, IC15 TPS7A2033PDBVR, IC9 TPS54060DGQ

Commit message: OSHW certification mark, front mask STEP color
Parts:
- C48, C52, C53: footprint PCM_EEZ_passives:C_1206_3216Metric -> PCM_EEZ_passives:C_0805_2012Metric; DigiKey 1276-2970-1-ND -> 1276-1244-1-ND; LCSC (none) -> C1779; Mouser 963-EMK316B7475ML-T -> 187-CL21A475KAQNNNE; TME GCM31CR71E475KA55L -> CL21A475KAQNNNE
Changed lines of the file:
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@@
 			)
 		)
-		(property "Footprint" "PCM_EEZ_passives:C_1206_3216Metric"
+		(property "Footprint" "PCM_EEZ_passives:C_0805_2012Metric"
 			(at 121.92 40.64 0)
 			(effects
@@
 			)
 		)
-		(property "DigiKey" "1276-2970-1-ND"
+		(property "DigiKey" "1276-1244-1-ND"
+			(at 121.92 43.18 0)
+			(effects
+				(font
+					(size 1.27 1.27)
+				)
+				(hide yes)
+			)
+		)
+		(property "Mouser" "187-CL21A475KAQNNNE"
 			(at 121.92 43.18 0)
 			(effects
@@
 			)
 		)
-		(property "Mouser" "963-EMK316B7475ML-T"
+		(property "TME" "CL21A475KAQNNNE"
 			(at 121.92 43.18 0)
 			(effects
@@
 			)
 		)
-		(property "TME" "GCM31CR71E475KA55L"
+		(property "LCSC" "C1779"
 			(at 121.92 43.18 0)
 			(effects
@@
 			)
 		)
-		(property "Footprint" "PCM_EEZ_passives:C_1206_3216Metric"
+		(property "Footprint" "PCM_EEZ_passives:C_0805_2012Metric"
 			(at 147.32 73.66 0)
 			(effects
@@
 			)
 		)
-		(property "DigiKey" "1276-2970-1-ND"
+		(property "DigiKey" "1276-1244-1-ND"
 			(at 147.32 76.2 0)
 			(effects
@@
 			)
 		)
-		(property "Mouser" "963-EMK316B7475ML-T"
+		(property "Mouser" "187-CL21A475KAQNNNE"
 			(at 147.32 76.2 0)
 			(effects
@@
 			)
 		)
-		(property "TME" "GCM31CR71E475KA55L"
+		(property "TME" "CL21A475KAQNNNE"
+			(at 147.32 76.2 0)
+			(effects
+				(font
+					(size 1.27 1.27)
+				)
+				(hide yes)
+			)
+		)
+		(property "LCSC" "C1779"
 			(at 147.32 76.2 0)
 			(effects
@@
 			)
 		)
-		(property "Footprint" "PCM_EEZ_passives:C_1206_3216Metric"
+		(property "Footprint" "PCM_EEZ_passives:C_0805_2012Metric"
 			(at 139.7 40.64 0)
 			(effects
@@
 			)
 		)
-		(property "DigiKey" "1276-2970-1-ND"
+		(property "DigiKey" "1276-1244-1-ND"
+			(at 139.7 43.18 0)
+			(effects
+				(font
+					(size 1.27 1.27)
+				)
+				(hide yes)
+			)
+		)
+		(property "Mouser" "187-CL21A475KAQNNNE"
 			(at 139.7 43.18 0)
 			(effects
@@
 			)
 		)
-		(property "Mouser" "963-EMK316B7475ML-T"
+		(property "TME" "CL21A475KAQNNNE"
 			(at 139.7 43.18 0)
 			(effects
@@
 			)
 		)
-		(property "TME" "GCM31CR71E475KA55L"
+		(property "LCSC" "C1779"
 			(at 139.7 43.18 0)
 			(effects

Commit message: JP3 update (Reset out select)
Parts:
- R30: value 6K2 -> 7K5
Changed lines of the file:
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@@
 	(title_block
 		(title "${project_name}")
-		(date "2026-02-12")
+		(date "2026-02-25")
 		(rev "${project_version}")
 		(company "${project_creator}")
@@
 			)
 		)
-		(property "Value" "6K2"
+		(property "Value" "7K5"
 			(at 133.35 93.345 0)
 			(effects
