File: KiCad/Bias_power.kicad_sch (KiCad schematic)
At the start: 42 parts, among them IC12 MC79L05, IC13 MC78L05, IC15 TPS7A2033PDBVR, IC9 TPS54060DGQ

Commit message: OSHWA logo added, KiCad 10 migration
Parts:
- JP6: value ~ -> (none)

Commit message: BOM and Gerbers update
Parts:
- C49: DigiKey (none) -> 1276-1101-1-ND; LCSC (none) -> C52306; Mouser (none) -> 187-CL32A226KAJNNNE; TME (none) -> CL32A226KAJNNNE
- D4, D5, D6, D7: LCSC (none) -> -
- FB2, FB3: LCSC (none) -> C337877
- R24, R26, R31: DigiKey (none) -> YAG1320CT-ND; LCSC (none) -> C859127; Mouser (none) -> 603-RC0805FR-0710RP
- R28: value 86K6 -> 51K; DigiKey 311-86.6KCRCT-ND -> 311-51.0KCRCT-ND; LCSC (none) -> C107233; Mouser 603-RT0805FRE0786K6L -> 603-RC0805FR-0751KL; TME CRCW080586K6FKTABC -> SMD0805-51K-1%
- R30: value 7K5 -> 4K7; DigiKey (none) -> 311-4.70KCRCT-ND; LCSC (none) -> C60816; Mouser (none) -> 603-RC0805FR-074K7L; TME (none) -> 0805S8F4701T5E
- TP3: Label -12V -> -VNR
- TP4: Label +12V -> +VNR
Other:
- note added: "+9.5 V"
- note added: "-9.5 V"
- note removed: "+12 V"
- note removed: "-12 V"
Changed lines of the file:
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@@
 		)
 	)
-	(text "-12 V"
+	(text "-9.5 V"
 		(exclude_from_sim no)
 		(at 134.62 38.1 0)
@@
 		)
 	)
-	(text "+12 V"
+	(text "+9.5 V"
 		(exclude_from_sim no)
 		(at 147.955 63.5 0)
@@
 			)
 		)
+		(property "LCSC" "-"
+			(at 101.6 71.12 90)
+			(hide yes)
+			(show_name no)
+			(do_not_autoplace no)
+			(effects
+				(font
+					(size 0.889 0.889)
+				)
+			)
+		)
 		(pin "A"
 		)
@@
 			)
 		)
-		(property "DigiKey" ""
+		(property "DigiKey" "1276-1101-1-ND"
 			(at 121.92 68.58 0)
 			(hide yes)
@@
 			)
 		)
-		(property "Mouser" ""
+		(property "Mouser" "187-CL32A226KAJNNNE"
 			(at 121.92 68.58 0)
 			(hide yes)
@@
 			)
 		)
-		(property "TME" ""
+		(property "TME" "CL32A226KAJNNNE"
 			(at 121.92 68.58 0)
 			(hide yes)
@@
 			)
 		)
-		(property "LCSC" ""
+		(property "LCSC" "C52306"
 			(at 121.92 68.58 0)
 			(hide yes)
@@
 			)
 		)
-		(property "LCSC" ""
+		(property "LCSC" "C337877"
 			(at 246.38 63.5 0)
 			(hide yes)
@@
 			)
 		)
-		(property "Value" "86K6"
+		(property "Value" "51K"
 			(at 133.35 77.47 0)
 			(show_name no)
@@
 			)
 		)
-		(property "DigiKey" "311-86.6KCRCT-ND "
+		(property "DigiKey" "311-51.0KCRCT-ND"
 			(at 132.08 76.2 0)
 			(hide yes)
@@
 			)
 		)
-		(property "Mouser" "603-RT0805FRE0786K6L "
+		(property "Mouser" "603-RC0805FR-0751KL"
 			(at 132.08 76.2 0)
 			(hide yes)
@@
 			)
 		)
-		(property "TME" "CRCW080586K6FKTABC"
+		(property "TME" "SMD0805-51K-1%"
 			(at 132.08 76.2 0)
 			(hide yes)
@@
 			)
 		)
+		(property "LCSC" "C107233"
+			(at 132.08 76.2 0)
+			(hide yes)
+			(show_name no)
+			(do_not_autoplace no)
+			(effects
+				(font
+					(size 0.889 0.889)
+				)
+			)
+		)
 		(pin "1"
 		)
@@
 			)
 		)
-		(property "Label" "-12V"
+		(property "Label" "-VNR"
 			(at 146.05 36.83 90)
+			(hide yes)
 			(show_name no)
 			(do_not_autoplace no)
@@
 			)
 		)
+		(property "DigiKey" "YAG1320CT-ND"
+			(at 114.3 68.58 0)
+			(hide yes)
+			(show_name no)
+			(do_not_autoplace no)
+			(effects
+				(font
+					(size 0.889 0.889)
+				)
+			)
+		)
+		(property "LCSC" "C859127"
+			(at 114.3 68.58 0)
+			(hide yes)
+			(show_name no)
+			(do_not_autoplace no)
+			(effects
+				(font
+					(size 0.889 0.889)
+				)
+			)
+		)
+		(property "Mouser" "603-RC0805FR-0710RP"
+			(at 114.3 68.58 0)
+			(hide yes)
+			(show_name no)
+			(do_not_autoplace no)
+			(effects
+				(font
+					(size 0.889 0.889)
+				)
+			)
+		)
 		(pin "1"
 		)
@@
 			)
 		)
+		(property "DigiKey" "YAG1320CT-ND"
+			(at 129.54 38.1 90)
+			(hide yes)
+			(show_name no)
+			(do_not_autoplace no)
+			(effects
+				(font
+					(size 0.889 0.889)
+				)
+			)
+		)
+		(property "LCSC" "C859127"
+			(at 129.54 38.1 90)
+			(hide yes)
+			(show_name no)
+			(do_not_autoplace no)
+			(effects
+				(font
+					(size 0.889 0.889)
+				)
+			)
+		)
+		(property "Mouser" "603-RC0805FR-0710RP"
+			(at 129.54 38.1 90)
+			(hide yes)
+			(show_name no)
+			(do_not_autoplace no)
+			(effects
+				(font
+					(size 0.889 0.889)
+				)
+			)
+		)
 		(pin "1"
 		)
@@
 			)
 		)
-		(property "Label" "+12V"
+		(property "Label" "+VNR"
 			(at 156.21 62.23 90)
+			(hide yes)
 			(show_name no)
 			(do_not_autoplace no)
@@
 			)
 		)
+		(property "LCSC" "-"
+			(at 111.76 38.1 0)
+			(hide yes)
+			(show_name no)
+			(do_not_autoplace no)
+			(effects
+				(font
+					(size 0.889 0.889)
+				)
+			)
+		)
 		(pin "A"
 		)
@@
 			)
 		)
+		(property "LCSC" "-"
+			(at 228.6 35.56 90)
+			(hide yes)
+			(show_name no)
+			(do_not_autoplace no)
+			(effects
+				(font
+					(size 0.889 0.889)
+				)
+			)
+		)
 		(pin "A"
 		)
@@
 			)
 		)
+		(property "LCSC" "-"
+			(at 228.6 68.58 90)
+			(hide yes)
+			(show_name no)
+			(do_not_autoplace no)
+			(effects
+				(font
+					(size 0.889 0.889)
+				)
+			)
+		)
 		(pin "A"
 		)
@@
 			)
 		)
-		(property "Value" "7K5"
+		(property "Value" "4K7"
 			(at 133.35 93.345 0)
 			(show_name no)
@@
 			)
 		)
-		(property "DigiKey" ""
+		(property "DigiKey" "311-4.70KCRCT-ND"
 			(at 132.08 91.44 0)
 			(hide yes)
@@
 			)
 		)
-		(property "Mouser" ""
+		(property "Mouser" "603-RC0805FR-074K7L"
 			(at 132.08 91.44 0)
 			(hide yes)
@@
 			)
 		)
-		(property "TME" ""
+		(property "TME" "0805S8F4701T5E"
 			(at 132.08 91.44 0)
 			(hide yes)
@@
 			)
 		)
-		(property "LCSC" ""
+		(property "LCSC" "C60816"
 			(at 132.08 91.44 0)
 			(hide yes)
@@
 			)
 		)
-		(property "LCSC" ""
+		(property "LCSC" "C337877"
 			(at 246.38 30.48 0)
 			(hide yes)
@@
 				)
 			)
+		)
+		(property "DigiKey" "YAG1320CT-ND"
+			(at 139.7 63.5 90)
+			(hide yes)
+			(show_name no)
+			(do_not_autoplace no)
+			(effects
+				(font
+					(size 0.889 0.889)
+				)
+			)
+		)
+		(property "LCSC" "C859127"
+			(at 139.7 63.5 90)
+			(hide yes)
+			(show_name no)
+			(do_not_autoplace no)
+			(effects
+				(font
+					(size 0.889 0.889)
+				)
+			)
+		)
+		(property "Mouser" "603-RC0805FR-0710RP"
+			(at 139.7 63.5 90)
+			(hide yes)
+			(show_name no)
+			(do_not_autoplace no)
+			(effects
+				(font
+					(size 0.889 0.889)
+				)
+			)

Commit message: #8, schematics annotated
Parts:
- renumbered R16 to R18, R17 to R19, R18 to R20, R20 to R22, R23 to R25, R24 to R26, R26 to R28, R28 to R30, R30 to R31, R31 to R33, TP3 to TP4, TP4 to TP5, TP5 to TP6, TP6 to TP7, TP7 to TP8
Changed lines of the file:
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@@
 	(title_block
 		(title "${project_name}")
-		(date "2026-05-10")
+		(date "2026-06-26")
 		(rev "${project_version}")
 		(company "${project_creator}")
@@
 		(in_pos_files yes)
 		(dnp no)
-		(property "Reference" "R28"
+		(property "Reference" "R30"
 			(at 133.35 75.565 0)
 			(show_name no)
@@
 			(project "EEZ DIB DCP405plus"
 				(path "/65943c0e-8943-4d2a-93dc-fb4938f73312/b522d90e-ad77-4f16-838a-4f8652a53e91"
-					(reference "R28")
+					(reference "R30")
 					(unit 1)
 				)
@@
 		(in_pos_files yes)
 		(dnp no)
-		(property "Reference" "TP3"
+		(property "Reference" "TP4"
 			(at 146.05 34.925 90)
 			(show_name no)
@@
 			(project "EEZ DIB DCP405plus"
 				(path "/65943c0e-8943-4d2a-93dc-fb4938f73312/b522d90e-ad77-4f16-838a-4f8652a53e91"
-					(reference "TP3")
+					(reference "TP4")
 					(unit 1)
 				)
@@
 		(in_pos_files yes)
 		(dnp no)
-		(property "Reference" "TP6"
+		(property "Reference" "TP7"
 			(at 234.95 57.15 90)
 			(show_name no)
@@
 			(project "EEZ DIB DCP405plus"
 				(path "/65943c0e-8943-4d2a-93dc-fb4938f73312/b522d90e-ad77-4f16-838a-4f8652a53e91"
-					(reference "TP6")
+					(reference "TP7")
 					(unit 1)
 				)
@@
 		(in_pos_files yes)
 		(dnp no)
-		(property "Reference" "#+3V09"
+		(property "Reference" "#+3V010"
 			(at 33.02 66.04 0)
 			(hide yes)
@@
 			(project "EEZ DIB DCP405plus"
 				(path "/65943c0e-8943-4d2a-93dc-fb4938f73312/b522d90e-ad77-4f16-838a-4f8652a53e91"
-					(reference "#+3V09")
+					(reference "#+3V010")
 					(unit 1)
 				)
@@
 		(in_pos_files yes)
 		(dnp no)
-		(property "Reference" "R24"
+		(property "Reference" "R26"
 			(at 113.03 68.58 0)
 			(show_name no)
@@
 			(project "EEZ DIB DCP405plus"
 				(path "/65943c0e-8943-4d2a-93dc-fb4938f73312/b522d90e-ad77-4f16-838a-4f8652a53e91"
-					(reference "R24")
+					(reference "R26")
 					(unit 1)
 				)
@@
 		(in_pos_files yes)
 		(dnp no)
-		(property "Reference" "R26"
+		(property "Reference" "R28"
 			(at 129.54 36.83 90)
 			(show_name no)
@@
 			(project "EEZ DIB DCP405plus"
 				(path "/65943c0e-8943-4d2a-93dc-fb4938f73312/b522d90e-ad77-4f16-838a-4f8652a53e91"
-					(reference "R26")
+					(reference "R28")
 					(unit 1)
 				)
@@
 		(in_pos_files yes)
 		(dnp no)
-		(property "Reference" "TP4"
+		(property "Reference" "TP5"
 			(at 156.21 60.325 90)
 			(show_name no)
@@
 			(project "EEZ DIB DCP405plus"
 				(path "/65943c0e-8943-4d2a-93dc-fb4938f73312/b522d90e-ad77-4f16-838a-4f8652a53e91"
-					(reference "TP4")
+					(reference "TP5")
 					(unit 1)
 				)
@@
 		(in_pos_files yes)
 		(dnp no)
-		(property "Reference" "#SUPPLY036"
+		(property "Reference" "#SUPPLY035"
 			(at 208.28 43.18 0)
 			(hide yes)
@@
 			(project "EEZ DIB DCP405plus"
 				(path "/65943c0e-8943-4d2a-93dc-fb4938f73312/b522d90e-ad77-4f16-838a-4f8652a53e91"
-					(reference "#SUPPLY036")
+					(reference "#SUPPLY035")
 					(unit 1)
 				)
@@
 		(in_pos_files yes)
 		(dnp no)
-		(property "Reference" "TP7"
+		(property "Reference" "TP8"
 			(at 245.11 100.33 90)
 			(show_name no)
@@
 			(project "EEZ DIB DCP405plus"
 				(path "/65943c0e-8943-4d2a-93dc-fb4938f73312/b522d90e-ad77-4f16-838a-4f8652a53e91"
-					(reference "TP7")
+					(reference "TP8")
 					(unit 1)
 				)
@@
 		(in_pos_files yes)
 		(dnp no)
-		(property "Reference" "R17"
+		(property "Reference" "R19"
 			(at 39.37 73.025 0)
 			(show_name no)
@@
 			(project "EEZ DIB DCP405plus"
 				(path "/65943c0e-8943-4d2a-93dc-fb4938f73312/b522d90e-ad77-4f16-838a-4f8652a53e91"
-					(reference "R17")
+					(reference "R19")
 					(unit 1)
 				)
@@
 		(in_pos_files yes)
 		(dnp no)
-		(property "Reference" "R23"
+		(property "Reference" "R25"
 			(at 87.63 86.36 0)
 			(show_name no)
@@
 			(project "EEZ DIB DCP405plus"
 				(path "/65943c0e-8943-4d2a-93dc-fb4938f73312/b522d90e-ad77-4f16-838a-4f8652a53e91"
-					(reference "R23")
+					(reference "R25")
 					(unit 1)
 				)
@@
 		(in_pos_files yes)
 		(dnp no)
-		(property "Reference" "R20"
+		(property "Reference" "R22"
 			(at 48.26 77.47 90)
 			(show_name no)
@@
 			(project "EEZ DIB DCP405plus"
 				(path "/65943c0e-8943-4d2a-93dc-fb4938f73312/b522d90e-ad77-4f16-838a-4f8652a53e91"
-					(reference "R20")
+					(reference "R22")
 					(unit 1)
 				)
@@
 		(in_pos_files yes)
 		(dnp no)
-		(property "Reference" "R18"
+		(property "Reference" "R20"
 			(at 45.72 62.23 90)
 			(show_name no)
@@
 			(project "EEZ DIB DCP405plus"
 				(path "/65943c0e-8943-4d2a-93dc-fb4938f73312/b522d90e-ad77-4f16-838a-4f8652a53e91"
-					(reference "R18")
+					(reference "R20")
 					(unit 1)
 				)
@@
 		(in_pos_files yes)
 		(dnp no)
-		(property "Reference" "R16"
+		(property "Reference" "R18"
 			(at 31.75 76.2 0)
 			(show_name no)
@@
 			(project "EEZ DIB DCP405plus"
 				(path "/65943c0e-8943-4d2a-93dc-fb4938f73312/b522d90e-ad77-4f16-838a-4f8652a53e91"
-					(reference "R16")
+					(reference "R18")
 					(unit 1)
 				)
@@
 		(in_pos_files yes)
 		(dnp no)
-		(property "Reference" "#SUPPLY035"
+		(property "Reference" "#SUPPLY034"
 			(at 205.74 121.92 0)
 			(hide yes)
@@
 			(project "EEZ DIB DCP405plus"
 				(path "/65943c0e-8943-4d2a-93dc-fb4938f73312/b522d90e-ad77-4f16-838a-4f8652a53e91"
-					(reference "#SUPPLY035")
+					(reference "#SUPPLY034")
 					(unit 1)
 				)
@@
 		(in_pos_files yes)
 		(dnp no)
-		(property "Reference" "TP5"
+		(property "Reference" "TP6"
 			(at 234.95 24.765 90)
 			(show_name no)
@@
 			(project "EEZ DIB DCP405plus"
 				(path "/65943c0e-8943-4d2a-93dc-fb4938f73312/b522d90e-ad77-4f16-838a-4f8652a53e91"
-					(reference "TP5")
+					(reference "TP6")
 					(unit 1)
 				)
@@
 		(in_pos_files yes)
 		(dnp no)
-		(property "Reference" "R30"
+		(property "Reference" "R31"
 			(at 133.35 91.44 0)
 			(show_name no)
@@
 			(project "EEZ DIB DCP405plus"
 				(path "/65943c0e-8943-4d2a-93dc-fb4938f73312/b522d90e-ad77-4f16-838a-4f8652a53e91"
-					(reference "R30")
+					(reference "R31")
 					(unit 1)
 				)
@@
 		(in_pos_files yes)
 		(dnp no)
-		(property "Reference" "#+3V017"
+		(property "Reference" "#+3V019"
 			(at 261.62 106.68 0)
 			(hide yes)
@@
 			(project "EEZ DIB DCP405plus"
 				(path "/65943c0e-8943-4d2a-93dc-fb4938f73312/b522d90e-ad77-4f16-838a-4f8652a53e91"
-					(reference "#+3V017")
+					(reference "#+3V019")
 					(unit 1)
 				)
@@
 		(in_pos_files yes)
 		(dnp no)
-		(property "Reference" "R31"
+		(property "Reference" "R33"
 			(at 139.7 62.23 90)
 			(show_name no)
@@
 			(project "EEZ DIB DCP405plus"
 				(path "/65943c0e-8943-4d2a-93dc-fb4938f73312/b522d90e-ad77-4f16-838a-4f8652a53e91"
-					(reference "R31")
+					(reference "R33")
 					(unit 1)
 				)
