File: KiCad/Bias_power.kicad_sch (KiCad schematic)
At the start: 42 parts, among them IC12 MC79L05, IC13 MC78L05, IC15 TPS7A2033PDBVR, IC9 TPS54060DGQ

Commit message: #9
Other:
- note added: "6K2???"

Commit message: Basic front mask gerbers, two test points, BOM updated
Parts:
- renumbered C36 to C112, C37 to C113, C38 to C114, C42 to C115, C43 to C116, C44 to C117, C46 to C118, C48 to C119, C49 to C120, C52 to C121, C53 to C122, C56 to C123, C58 to C124, C59 to C125, C60 to C126, D4 to D20, D5 to D21, D6 to D22, D7 to D23, IC9 to IC24, IC12 to IC25, IC13 to IC26, IC15 to IC27, JP6 to JP14, R18 to R142, R19 to R143, R20 to R144, R22 to R145, R25 to R146, R26 to R147, R28 to R148, R30 to R149, R31 to R150, R33 to R151, TP4 to TP14, TP5 to TP15, TP6 to TP16, TP7 to TP17, TP8 to TP18, TR1 to TR2

Commit message: ADC DRDY test point added
Parts:
- renumbered TP14 to TP15, TP15 to TP16, TP16 to TP17, TP17 to TP18, TP18 to TP19
Changed lines of the file:
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@@
 	(title_block
 		(title "${project_name}")
-		(date "2026-09-20")
+		(date "2026-09-21")
 		(rev "${project_version}")
 		(company "${project_creator}")
@@
 		(in_pos_files no)
 		(dnp no)
-		(property "Reference" "TP14"
+		(property "Reference" "TP15"
 			(at 146.05 34.925 90)
 			(show_name no)
@@
 			(project "EEZ DIB DCP405plus"
 				(path "/65943c0e-8943-4d2a-93dc-fb4938f73312/b522d90e-ad77-4f16-838a-4f8652a53e91"
-					(reference "TP14")
+					(reference "TP15")
 					(unit 1)
 				)
@@
 		(in_pos_files no)
 		(dnp no)
-		(property "Reference" "TP17"
+		(property "Reference" "TP18"
 			(at 234.95 57.15 90)
 			(show_name no)
@@
 			(project "EEZ DIB DCP405plus"
 				(path "/65943c0e-8943-4d2a-93dc-fb4938f73312/b522d90e-ad77-4f16-838a-4f8652a53e91"
-					(reference "TP17")
+					(reference "TP18")
 					(unit 1)
 				)
@@
 		(in_pos_files no)
 		(dnp no)
-		(property "Reference" "TP15"
+		(property "Reference" "TP16"
 			(at 156.21 60.325 90)
 			(show_name no)
@@
 			(project "EEZ DIB DCP405plus"
 				(path "/65943c0e-8943-4d2a-93dc-fb4938f73312/b522d90e-ad77-4f16-838a-4f8652a53e91"
-					(reference "TP15")
+					(reference "TP16")
 					(unit 1)
 				)
@@
 		(in_pos_files no)
 		(dnp no)
-		(property "Reference" "TP18"
+		(property "Reference" "TP19"
 			(at 245.11 100.33 90)
 			(show_name no)
@@
 			(project "EEZ DIB DCP405plus"
 				(path "/65943c0e-8943-4d2a-93dc-fb4938f73312/b522d90e-ad77-4f16-838a-4f8652a53e91"
-					(reference "TP18")
+					(reference "TP19")
 					(unit 1)
 				)
@@
 		(in_pos_files no)
 		(dnp no)
-		(property "Reference" "TP16"
+		(property "Reference" "TP17"
 			(at 234.95 24.765 90)
 			(show_name no)
@@
 			(project "EEZ DIB DCP405plus"
 				(path "/65943c0e-8943-4d2a-93dc-fb4938f73312/b522d90e-ad77-4f16-838a-4f8652a53e91"
-					(reference "TP16")
+					(reference "TP17")
 					(unit 1)
 				)

Commit message: #10
Parts:
- renumbered TP15 to TP14, TP16 to TP15, TP17 to TP16, TP18 to TP17, TP19 to TP18
Changed lines of the file:
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@@
 	(title_block
 		(title "${project_name}")
-		(date "2026-09-21")
+		(date "2026-10-08")
 		(rev "${project_version}")
 		(company "${project_creator}")
@@
 		(in_pos_files no)
 		(dnp no)
-		(property "Reference" "TP15"
+		(property "Reference" "TP14"
 			(at 146.05 34.925 90)
 			(show_name no)
@@
 			(project "EEZ DIB DCP405plus"
 				(path "/65943c0e-8943-4d2a-93dc-fb4938f73312/b522d90e-ad77-4f16-838a-4f8652a53e91"
-					(reference "TP15")
+					(reference "TP14")
 					(unit 1)
 				)
@@
 		(in_pos_files no)
 		(dnp no)
-		(property "Reference" "TP18"
+		(property "Reference" "TP17"
 			(at 234.95 57.15 90)
 			(show_name no)
@@
 			(project "EEZ DIB DCP405plus"
 				(path "/65943c0e-8943-4d2a-93dc-fb4938f73312/b522d90e-ad77-4f16-838a-4f8652a53e91"
-					(reference "TP18")
+					(reference "TP17")
 					(unit 1)
 				)
@@
 		(in_pos_files no)
 		(dnp no)
-		(property "Reference" "TP16"
+		(property "Reference" "TP15"
 			(at 156.21 60.325 90)
 			(show_name no)
@@
 			(project "EEZ DIB DCP405plus"
 				(path "/65943c0e-8943-4d2a-93dc-fb4938f73312/b522d90e-ad77-4f16-838a-4f8652a53e91"
-					(reference "TP16")
+					(reference "TP15")
 					(unit 1)
 				)
@@
 		(in_pos_files no)
 		(dnp no)
-		(property "Reference" "TP19"
+		(property "Reference" "TP18"
 			(at 245.11 100.33 90)
 			(show_name no)
@@
 			(project "EEZ DIB DCP405plus"
 				(path "/65943c0e-8943-4d2a-93dc-fb4938f73312/b522d90e-ad77-4f16-838a-4f8652a53e91"
-					(reference "TP19")
+					(reference "TP18")
 					(unit 1)
 				)
@@
 		(in_pos_files no)
 		(dnp no)
-		(property "Reference" "TP17"
+		(property "Reference" "TP16"
 			(at 234.95 24.765 90)
 			(show_name no)
@@
 			(project "EEZ DIB DCP405plus"
 				(path "/65943c0e-8943-4d2a-93dc-fb4938f73312/b522d90e-ad77-4f16-838a-4f8652a53e91"
-					(reference "TP17")
+					(reference "TP16")
 					(unit 1)
 				)
