File: KiCad/CC_CV_OVP.kicad_sch (KiCad schematic)
At the start: 41 parts, among them IC26 LM293D, IC27 MAX9141ESA, Q25 2N7002, Q26 2N7002, Q27 2N7002, Q28 MMBT5551, Q29 FMMT493TA, Q30 BT139B-600E, Q31 PSMN013-60YL

Commit message: Gerbers update
Parts:
- renumbered C123 to C122, C124 to C123, C125 to C124, C126 to C125, C127 to C126, ZD7 to ZD8
Changed lines of the file:
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@@
 	(title_block
 		(title "${project_name}")
-		(date "2026-01-06")
+		(date "2026-01-13")
 		(rev "${project_version}")
 		(company "${project_creator}")
@@
 		(on_board yes)
 		(dnp no)
-		(property "Reference" "C125"
+		(property "Reference" "C124"
 			(at 183.134 64.516 0)
 			(effects
@@
 			(project "EEZ DIB DCP405"
 				(path "/65943c0e-8943-4d2a-93dc-fb4938f73312/5aca86d7-0c45-458c-9a52-ab1a5068ba91"
-					(reference "C125")
+					(reference "C124")
 					(unit 1)
 				)
@@
 		(on_board yes)
 		(dnp no)
-		(property "Reference" "C123"
+		(property "Reference" "C122"
 			(at 121.539 58.039 90)
 			(effects
@@
 			(project "EEZ DIB DCP405"
 				(path "/65943c0e-8943-4d2a-93dc-fb4938f73312/5aca86d7-0c45-458c-9a52-ab1a5068ba91"
-					(reference "C123")
+					(reference "C122")
 					(unit 1)
 				)
@@
 		(on_board yes)
 		(dnp no)
-		(property "Reference" "C126"
+		(property "Reference" "C125"
 			(at 190.119 41.021 90)
 			(effects
@@
 			(project "EEZ DIB DCP405"
 				(path "/65943c0e-8943-4d2a-93dc-fb4938f73312/5aca86d7-0c45-458c-9a52-ab1a5068ba91"
-					(reference "C126")
+					(reference "C125")
 					(unit 1)
 				)
@@
 		(on_board yes)
 		(dnp no)
-		(property "Reference" "ZD7"
+		(property "Reference" "ZD8"
 			(at 241.935 93.98 90)
 			(effects
@@
 			(project "EEZ DIB DCP405"
 				(path "/65943c0e-8943-4d2a-93dc-fb4938f73312/5aca86d7-0c45-458c-9a52-ab1a5068ba91"
-					(reference "ZD7")
+					(reference "ZD8")
 					(unit 1)
 				)
@@
 		(on_board yes)
 		(dnp no)
-		(property "Reference" "C124"
+		(property "Reference" "C123"
 			(at 121.539 73.279 90)
 			(effects
@@
 			(project "EEZ DIB DCP405"
 				(path "/65943c0e-8943-4d2a-93dc-fb4938f73312/5aca86d7-0c45-458c-9a52-ab1a5068ba91"
-					(reference "C124")
+					(reference "C123")
 					(unit 1)
 				)
@@
 		(on_board yes)
 		(dnp no)
-		(property "Reference" "C127"
+		(property "Reference" "C126"
 			(at 193.294 107.696 0)
 			(effects
@@
 			(project "EEZ DIB DCP405"
 				(path "/65943c0e-8943-4d2a-93dc-fb4938f73312/5aca86d7-0c45-458c-9a52-ab1a5068ba91"
-					(reference "C127")
+					(reference "C126")
 					(unit 1)
 				)
