File: KiCad/CC_CV_OVP.kicad_sch (KiCad schematic)
At the start: 41 parts, among them IC26 LM293D, IC27 MAX9141ESA, Q25 2N7002, Q26 2N7002, Q27 2N7002, Q28 MMBT5551, Q29 FMMT493TA, Q30 BT139B-600E, Q31 PSMN013-60YL

Commit message: BOM and Gerbers update
Parts:
- D22, D23: LCSC (none) -> C109218
- R124, R125: DigiKey (none) -> 311-6.20KCRCT-ND; LCSC (none) -> C114535; Mouser (none) -> 603-RC0805FR-076K2L; TME (none) -> -
- R134: LCSC (none) -> C60816
Changed lines of the file:
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@@
 			)
 		)
+		(property "DigiKey" "311-6.20KCRCT-ND"
+			(at 53.34 86.36 90)
+			(hide yes)
+			(show_name no)
+			(do_not_autoplace no)
+			(effects
+				(font
+					(size 0.889 0.889)
+				)
+			)
+		)
+		(property "LCSC" "C114535"
+			(at 53.34 86.36 90)
+			(hide yes)
+			(show_name no)
+			(do_not_autoplace no)
+			(effects
+				(font
+					(size 0.889 0.889)
+				)
+			)
+		)
+		(property "Mouser" "603-RC0805FR-076K2L"
+			(at 53.34 86.36 90)
+			(hide yes)
+			(show_name no)
+			(do_not_autoplace no)
+			(effects
+				(font
+					(size 0.889 0.889)
+				)
+			)
+		)
+		(property "TME" "-"
+			(at 53.34 86.36 90)
+			(hide yes)
+			(show_name no)
+			(do_not_autoplace no)
+			(effects
+				(font
+					(size 0.889 0.889)
+				)
+			)
+		)
 		(pin "1"
 		)
@@
 			)
 		)
+		(property "DigiKey" "311-6.20KCRCT-ND"
+			(at 53.34 45.72 90)
+			(hide yes)
+			(show_name no)
+			(do_not_autoplace no)
+			(effects
+				(font
+					(size 0.889 0.889)
+				)
+			)
+		)
+		(property "LCSC" "C114535"
+			(at 53.34 45.72 90)
+			(hide yes)
+			(show_name no)
+			(do_not_autoplace no)
+			(effects
+				(font
+					(size 0.889 0.889)
+				)
+			)
+		)
+		(property "Mouser" "603-RC0805FR-076K2L"
+			(at 53.34 45.72 90)
+			(hide yes)
+			(show_name no)
+			(do_not_autoplace no)
+			(effects
+				(font
+					(size 0.889 0.889)
+				)
+			)
+		)
+		(property "TME" "-"
+			(at 53.34 45.72 90)
+			(hide yes)
+			(show_name no)
+			(do_not_autoplace no)
+			(effects
+				(font
+					(size 0.889 0.889)
+				)
+			)
+		)
 		(pin "1"
 		)
@@
 			)
 		)
+		(property "LCSC" "C109218"
+			(at 228.6 76.2 90)
+			(hide yes)
+			(show_name no)
+			(do_not_autoplace no)
+			(effects
+				(font
+					(size 0.889 0.889)
+				)
+			)
+		)
 		(pin "A"
 		)
@@
 			)
 		)
+		(property "LCSC" "C60816"
+			(at 200.66 109.22 0)
+			(hide yes)
+			(show_name no)
+			(do_not_autoplace no)
+			(effects
+				(font
+					(size 0.889 0.889)
+				)
+			)
+		)
 		(pin "1"
 		)
@@
 				)
 			)
+		)
+		(property "LCSC" "C109218"
+			(at 228.6 68.58 90)
+			(hide yes)
+			(show_name no)
+			(do_not_autoplace no)
+			(effects
+				(font
+					(size 0.889 0.889)
+				)
+			)

Commit message: #8, schematics annotated
Parts:
- renumbered LED3 to LED4, Q25 to Q23, Q26 to Q24, Q27 to Q25, Q28 to Q26, Q29 to Q27, Q30 to Q28, Q31 to Q29, R122 to R130, R123 to R131, R124 to R132, R125 to R133, R126 to R134, R127 to R135, R128 to R136, R129 to R137, R130 to R138, R131 to R139, R132 to R140, R133 to R141, R134 to R142, R135 to R143, R136 to R144, R137 to R145, R138 to R146, R139 to R147, R140 to R148, R141 to R149, R142 to R150, R143 to R151
