File: KiCad/CC_CV_OVP.kicad_sch (KiCad schematic)
At the start: 41 parts, among them IC26 LM293D, IC27 MAX9141ESA, Q23 2N7002, Q24 2N7002, Q25 2N7002, Q26 MMBT5551, Q27 FMMT493TA, Q28 BT139B-600E, Q29 PSMN013-60YL

Commit message: #9
Parts:
- ZD8: Label (none) -> 4.7V

Commit message: Basic front mask gerbers, two test points, BOM updated
Parts:
- renumbered C122 to C107, C123 to C108, C124 to C109, C125 to C110, C126 to C111, D22 to D18, D23 to D19, IC26 to IC22, IC27 to IC23, JP12 to JP13, R130 to R120, R131 to R121, R132 to R122, R133 to R123, R134 to R124, R135 to R125, R136 to R126, R137 to R127, R138 to R128, R139 to R129, R140 to R130, R141 to R131, R142 to R132, R143 to R133, R144 to R134, R145 to R135, R146 to R136, R147 to R137, R148 to R138, R149 to R139, R150 to R140, R151 to R141
