File: KiCad/Post-regulator.kicad_sch (KiCad schematic)
At the start: 105 parts, among them IC17 LTC2050HVCS8#PBF, IC18 TL072D, IC19 TL072D, IC20 SN74LVC1G3157DCKR, Q10 MMBT5401, Q11 MMBT5401, Q12 BCP56-16.115, Q13 MMBT5551, Q14 IRFP250NPBF, Q15 BCP56-16.115, Q16 BC857C, Q17 IRFI9Z34GPBF, Q18 PSMN0R9-25YLC, Q19 PSMN0R9-25YLC, Q9 MMBT5551

Commit message: #4
Parts:
- removed KK10: B3/BN2842, symbol PCM_EEZ_unsorted:B3/BN2842
- removed KK9: M3X8/D7985B, symbol PCM_EEZ_unsorted:M3X8/D7985B
Changed lines of the file:
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@@
 	(title_block
 		(title "${project_name}")
-		(date "2026-03-05")
+		(date "2026-03-22")
 		(rev "${project_version}")
 		(company "${project_creator}")
@@
 	)
 	(symbol
-		(lib_id "PCM_EEZ_unsorted:M3X8/D7985B")
-		(at 182.88 58.42 0)
-		(unit 1)
-		(exclude_from_sim no)
-		(in_bom yes)
-		(on_board no)
-		(dnp no)
-		(fields_autoplaced yes)
-		(property "Reference" "KK9"
-			(at 185.42 58.42 0)
-			(do_not_autoplace yes)
-			(effects
-				(font
-					(size 1.27 1.27)
-				)
-				(justify left bottom)
-			)
-		)
-		(property "Value" "M3X8/D7985B"
-			(at 185.42 60.325 0)
-			(do_not_autoplace yes)
-			(effects
-				(font
-					(size 1.27 1.27)
-				)
-				(justify left bottom)
-			)
-		)
-		(property "Footprint" ""
-			(at 182.88 58.42 0)
-			(effects
-				(font
-					(size 1.27 1.27)
-				)
-				(hide yes)
-			)
-		)
-		(property "Datasheet" ""
-			(at 182.88 58.42 0)
-			(effects
-				(font
-					(size 1.27 1.27)
-				)
-				(hide yes)
-			)
-		)
-		(property "Description" "Screw; M3x8; 0.5; Head: cheese head; Phillips; PH1; DIN 7985"
-			(at 182.88 60.96 0)
-			(effects
-				(font
-					(size 1.27 1.27)
-				)
-				(hide yes)
-			)
-		)
-		(property "DigiKey" "-"
-			(at 182.88 63.5 0)
-			(show_name yes)
-			(effects
-				(font
-					(size 1.27 1.27)
-				)
-				(hide yes)
-			)
-		)
-		(property "Mouser" "-"
-			(at 182.88 66.04 0)
-			(show_name yes)
-			(effects
-				(font
-					(size 1.27 1.27)
-				)
-				(hide yes)
-			)
-		)
-		(property "TME" "M3X8/D7985B"
-			(at 182.88 68.58 0)
-			(show_name yes)
-			(effects
-				(font
-					(size 1.27 1.27)
-				)
-				(hide yes)
-			)
-		)
-		(instances
-			(project "EEZ DIB DCP405plus"
-				(path "/65943c0e-8943-4d2a-93dc-fb4938f73312/34bb83a5-d559-4d80-b3e4-82ef079c17b9"
-					(reference "KK9")
-					(unit 1)
-				)
-			)
-		)
-	)
-	(symbol
 		(lib_id "PCM_EEZ_passives:C-EU")
 		(at 132.08 149.86 270)
@@
 					(unit 1)
 				)
-			)
-		)
-	)
-	(symbol
-		(lib_id "PCM_EEZ_unsorted:B3/BN2842")
-		(at 183.515 53.34 0)
-		(unit 1)
-		(exclude_from_sim no)
-		(in_bom yes)
-		(on_board no)
-		(dnp no)
-		(property "Reference" "KK10"
-			(at 185.42 53.34 0)
-			(do_not_autoplace yes)
-			(effects
-				(font
-					(size 1.27 1.27)
-				)
-				(justify left bottom)
-			)
-		)
-		(property "Value" "B3/BN2842"
-			(at 185.42 55.245 0)
-			(do_not_autoplace yes)
-			(effects
-				(font
-					(size 1.27 1.27)
-				)
-				(justify left bottom)
-			)
-		)
-		(property "Footprint" ""
-			(at 183.515 53.34 0)
-			(effects
-				(font
-					(size 1.27 1.27)
-				)
-				(hide yes)
-			)
-		)
-		(property "Datasheet" ""
-			(at 183.515 53.34 0)
-			(effects
-				(font
-					(size 1.27 1.27)
-				)
-				(hide yes)
-			)
-		)
-		(property "Description" "Washer; externally serrated; M3"
-			(at 183.515 55.88 0)
-			(effects
-				(font
-					(size 1.27 1.27)
-				)
-				(hide yes)
-			)
-		)
-		(property "DigiKey" "-"
-			(at 183.515 58.42 0)
-			(show_name yes)
-			(effects
-				(font
-					(size 1.27 1.27)
-				)
-				(hide yes)
-			)
-		)
-		(property "Mouser" "-"
-			(at 183.515 60.96 0)
-			(show_name yes)
-			(effects
-				(font
-					(size 1.27 1.27)
-				)
-				(hide yes)
-			)
-		)
-		(property "TME" "B3/BN2842"
-			(at 183.515 63.5 0)
-			(show_name yes)
-			(effects
-				(font
-					(size 1.27 1.27)
-				)
-				(hide yes)
-			)
-		)
-		(instances
-			(project "EEZ DIB DCP405plus"
-				(path "/65943c0e-8943-4d2a-93dc-fb4938f73312/34bb83a5-d559-4d80-b3e4-82ef079c17b9"
-					(reference "KK10")
-					(unit 1)
-				)
