File: KiCad/Post-regulator.kicad_sch (KiCad schematic)
At the start: 103 parts, among them IC17 LTC2050HVCS8#PBF, IC18 TL072D, IC19 TL072D, IC20 SN74LVC1G3157DCKR, Q10 MMBT5401, Q11 MMBT5401, Q12 BCP56-16.115, Q13 MMBT5551, Q14 IRFP250NPBF, Q15 BCP56-16.115, Q16 BC857C, Q17 IRFI9Z34GPBF, Q18 PSMN0R9-25YLC, Q19 PSMN0R9-25YLC, Q9 MMBT5551

Commit message: Basic variant schematics PDF
Other:
- note added: "FS: 124K / 7.5K = 16.534 * 2.5 = 41.34 V Zero offset: 16.534 * 0.05 = 0.8267 V"
- note added: "FS: 750R / 30K: x40 = 6.25 A FS: 750R / 30.1K: x40.133 = 6.23 A FS: 750R / 36K: x48 = 5.208 A Zero offset: 0.75/36 = 0.020834 * 0.05 / 0.01 = 0.1042 V"
- note added: "Note 3.1: Q14, Q17 and R77 (if used) mounted on heatsink KK7 Note 3.2: Use power resistors with the lowest possible TCR (below ± 50 ppm/oC), e.g. GMR100HJBFA10L0"
- note removed: "750R / 30K: x40 ... 6.25 A full scale 750R / 30.1K: x40.133 ... 6.23 A full scale 750R / 36K: x48 ... 5.208 A full scale"
- note removed: "Note 3.1: Q12, Q15 and R79 (if used) mounted on heatsink KK3 Note 3.2: Use power resistors with the lowest possible TCR (below ± 50 ppm/oC), e.g. GMR100HJBFA10L0"
Changed lines of the file:
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@@
 	(title_block
 		(title "${project_name}")
-		(date "2026-04-30")
+		(date "2026-05-10")
 		(rev "${project_version}")
 		(company "${project_creator}")
@@
 		)
 	)
+	(text "FS: 124K / 7.5K = 16.534 * 2.5 = 41.34 V\nZero offset: 16.534 * 0.05 = 0.8267 V"
+		(exclude_from_sim no)
+		(at 216.535 99.06 0)
+		(effects
+			(font
+				(size 0.889 0.889)
+				(color 132 0 132 1)
+			)
+			(justify left top)
+		)
+	)
 	(text "11K"
 		(exclude_from_sim no)
@@
 		)
 	)
-	(text "750R / 30K: x40 ... 6.25 A full scale\n750R / 30.1K: x40.133 ... 6.23 A full scale\n750R / 36K: x48 ... 5.208 A full scale"
-		(exclude_from_sim no)
-		(at 144.78 180.34 0)
-		(effects
-			(font
-				(size 0.889 0.889)
-				(color 255 0 0 1)
+	(text "FS: 750R / 30K: x40 = 6.25 A\nFS: 750R / 30.1K: x40.133 = 6.23 A\nFS: 750R / 36K: x48 = 5.208 A\n\nZero offset: 0.75/36 = 0.020834 * 0.05 / 0.01 = 0.1042 V"
+		(exclude_from_sim no)
+		(at 130.81 178.435 0)
+		(effects
+			(font
+				(size 0.889 0.889)
+				(color 132 0 132 1)
 			)
 			(justify left top)
 		)
 	)
-	(text "Note 3.1: Q12, Q15 and R79 (if used) mounted on heatsink KK3\nNote 3.2: Use power resistors with the lowest possible TCR (below ± 50 ppm/oC), e.g. GMR100HJBFA10L0"
+	(text "Note 3.1: Q14, Q17 and R77 (if used) mounted on heatsink KK7\nNote 3.2: Use power resistors with the lowest possible TCR (below ± 50 ppm/oC), e.g. GMR100HJBFA10L0"
 		(exclude_from_sim no)
 		(at 17.78 193.04 0)

Commit message: BOM and Gerbers update
Parts:
- C100, C99: LCSC (none) -> C307541; TME (none) -> CL21B222JBANNNC
- D11, D12, D13, D14, D15, D16, D17, D18: LCSC (none) -> C109218
- R49: DigiKey (none) -> YAG1320CT-ND; LCSC (none) -> C859127; Mouser (none) -> 603-RC0805FR-0710RP
- R50: DigiKey (none) -> 311-1.20KCRCT-ND; LCSC (none) -> C114526; Mouser (none) -> 603-RC0805FR-071K2L; TME (none) -> SMD0805-1K2-1%
- R53: DigiKey (none) -> 311-51.0KCRCT-ND; LCSC (none) -> C107233; Mouser (none) -> 603-RC0805FR-0751KL; TME (none) -> SMD0805-51K-1%
- R59: DigiKey (none) -> 311-16.0KCRCT-ND; LCSC (none) -> C137588; Mouser (none) -> 603-RC0805FR-0716KL; TME (none) -> SMD0805-16K-1%
- R68: DigiKey (none) -> 311-6.80KCRCT-ND; LCSC (none) -> C114550; Mouser (none) -> 603-RC0805FR-076K8L; TME (none) -> SMD0805-6K8-1%
- R69: DigiKey (none) -> 311-3.00KCRCT-ND; LCSC (none) -> C126350; Mouser (none) -> 603-RC0805FR-073KL; TME (none) -> SMD0805-3K-1%
- R75: DigiKey (none) -> 311-6.20KCRCT-ND; LCSC (none) -> C114535; Mouser (none) -> 603-RC0805FR-076K2L; TME (none) -> -
- R86, R87: DigiKey (none) -> YAG4808CT-ND; LCSC (none) -> C122537; Mouser (none) -> 603-RT0805BRB07100KL; TME (none) -> RT0805BRD07100KL
- R91, R92: DigiKey (none) -> P24KBFCT-ND; LCSC (none) -> C136924; Mouser (none) -> 667-ERA-6ARB243V; TME (none) -> -

Commit message: #8, schematics annotated
Parts:
- renumbered Q12 to Q10, Q13 to Q11, Q14 to Q12, Q15 to Q13, Q16 to Q14, Q17 to Q15, Q18 to Q16, Q19 to Q17, Q9 to Q7, Q10 to Q8, Q11 to Q9, R97 to R100, R98 to R101, R49 to R52, R50 to R53, R51 to R54, R52 to R55, R53 to R56, R54 to R57, R55 to R58, R56 to R59, R57 to R60, R58 to R61, R59 to R62, R60 to R63, R61 to R64, R62 to R65, R63 to R66, R64 to R67, R65 to R68, R66 to R69, R67 to R70, R68 to R71, R69 to R72, R70 to R73, R71 to R74, R72 to R75, R73 to R76, R74 to R77, R75 to R78, R76 to R79, R77 to R80, R78 to R81, R79 to R82, R80 to R83, R81 to R84, R82 to R85, R83 to R86, R84 to R87, R85 to R88, R86 to R89, R87 to R90, R88 to R91, R89 to R92, R90 to R93, R91 to R94, R92 to R95, R93 to R96, R94 to R97, R95 to R98, R96 to R99
