File: KiCad/Post-regulator.kicad_sch (KiCad schematic)
At the start: 103 parts, among them IC17 LTC2050HVCS8#PBF, IC18 TL072D, IC19 TL072D, IC20 SN74LVC1G3157DCKR, Q10 BCP56-16.115, Q11 MMBT5551, Q12 IRFP250NPBF, Q13 BCP56-16.115, Q14 BC857C, Q15 IRFI9Z34GPBF, Q16 PSMN0R9-25YLC, Q17 PSMN0R9-25YLC, Q7 MMBT5551, Q8 MMBT5401, Q9 MMBT5401

Commit message: #9
Other:
- note added: "36K5 0.1%"

Commit message: Basic front mask gerbers, two test points, BOM updated
Parts:
- D15: renamed from D19; now in the parts list
- renumbered C84 to C69, C85 to C70, C86 to C71, C87 to C72, C88 to C73, C89 to C74, C90 to C75, C91 to C76, C92 to C77, C93 to C78, C94 to C79, C95 to C80, C96 to C81, C97 to C82, C98 to C83, C99 to C84, C100 to C85, C101 to C86, C102 to C87, C103 to C88, C104 to C89, C105 to C90, C106 to C91, C107 to C92, C108 to C93, D14 to D10, D15 to D11, D16 to D12, D17 to D13, D18 to D14, D11 to D7, D12 to D8, D13 to D9, IC17 to IC13, IC18 to IC14, IC19 to IC15, IC20 to IC16, R52 to R42, R53 to R43, R54 to R44, R55 to R45, R56 to R46, R57 to R47, R58 to R48, R59 to R49, R60 to R50, R61 to R51, R62 to R52, R63 to R53, R64 to R54, R65 to R55, R66 to R56, R67 to R57, R68 to R58, R69 to R59, R70 to R60, R71 to R61, R72 to R62, R73 to R63, R74 to R64, R75 to R65, R76 to R66, R77 to R67, R78 to R68, R79 to R69, R80 to R70, R81 to R71, R82 to R72, R83 to R73, R84 to R74, R85 to R75, R86 to R76, R87 to R77, R88 to R78, R89 to R79, R90 to R80, R91 to R81, R92 to R82, R93 to R83, R94 to R84, R95 to R85, R96 to R86, R97 to R87, R98 to R88, R99 to R89, R100 to R90, R101 to R91
