File: KiCad/Power_pre-regulator.kicad_sch (KiCad schematic)
At the start: 65 parts, among them IC16 LM5145RGYR, Q4 BSC117N08NS5ATMA1, Q5 BSC039N06NSATMA1, Q6 2N7002, Q7 MMBT5401, Q8 DMP6023LFG-7, X3 B4P-VH (LF)(SN)

Commit message: X3 type changed
Parts:
- X3: value B4P-VH (LF)(SN) -> B4PS-VH (LF)(SN); footprint PCM_EEZ_connectors:B4P-VH_LF_SN -> PCM_EEZ_connectors:B4PS-VH; DigiKey (none) -> 455-B4PS-VH-ND; Mouser (none) -> 306-B4PS-VHLFSN; TME B4P-VH (LF)(SN) -> B4PS-VH (LF)(SN)
Changed lines of the file:
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@@
 	(title_block
 		(title "${project_name}")
-		(date "2025-12-18")
+		(date "2026-01-03")
 		(rev "${project_version}")
 		(company "${project_creator}")
@@
 			)
 		)
-		(property "Value" "B4P-VH (LF)(SN)"
+		(property "Value" "B4PS-VH (LF)(SN)"
 			(at 25.4 37.465 0)
 			(effects
@@
 			)
 		)
-		(property "Footprint" "PCM_EEZ_connectors:B4P-VH_LF_SN"
+		(property "Footprint" "PCM_EEZ_connectors:B4PS-VH"
 			(at 25.4 33.02 0)
 			(effects
@@
 			)
 		)
-		(property "DigiKey" ""
+		(property "DigiKey" "455-B4PS-VH-ND"
 			(at 25.4 33.02 0)
 			(effects
@@
 			)
 		)
-		(property "Mouser" ""
+		(property "Mouser" "306-B4PS-VHLFSN"
 			(at 25.4 33.02 0)
 			(effects
@@
 			)
 		)
-		(property "TME" "B4P-VH (LF)(SN)"
+		(property "TME" "B4PS-VH (LF)(SN)"
 			(at 25.4 33.02 0)
 			(effects

Commit message: Gerbers update
Parts:
- removed C79: 10n, PCM_EEZ_passives:C_0805_2012Metric, symbol PCM_EEZ_passives:C-EU
- added ZD3: BZX384-C15, PCM_EEZ_SMD:SOD-323_1P8X1P35_ONS-M, symbol PCM_EEZ_discretes:DIODE_ZENER
- Q8: value DMP6023LFG-7 -> SQJ457EP-T1_BE3; footprint PCM_EEZ_SMD:TRANS_FDMC8010 -> PCM_EEZ_SMD:PowerPAK SO-8; DigiKey DMP6023LFG-7DICT-ND -> 742-SQJ457EP-T1_BE3CT-ND; LCSC C526579 -> C7364386; Mouser 621-DMP6023LFG-7 -> 78-SQJ457EP-T1_BE3
- renumbered C80 to C79, C81 to C80, C82 to C81, C83 to C82, C84 to C83
Connections:
- net DC_OUT: now also ZD3.C
- net at Q6.3 (D), Q8.4 (G), R42.1: now also ZD3.A
Changed lines of the file:
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@@
 	(title_block
 		(title "${project_name}")
-		(date "2026-01-06")
+		(date "2026-01-13")
 		(rev "${project_version}")
 		(company "${project_creator}")
@@
 	(text "100% Duty"
 		(exclude_from_sim no)
-		(at 195.58 33.02 0)
+		(at 193.04 33.02 0)
 		(effects
 			(font
@@
 	(wire
 		(pts
+			(xy 203.2 35.56) (xy 203.2 38.1)
+		)
+		(stroke
+			(width 0)
+			(type default)
+		)
+	)
+	(wire
+		(pts
 			(xy 198.12 99.06) (xy 198.12 91.44)
 		)
@@
 	(polyline
 		(pts
-			(xy 238.76 27.94) (xy 193.04 27.94)
+			(xy 238.76 27.94) (xy 190.5 27.94)
 		)
 		(stroke
@@
 	(polyline
 		(pts
-			(xy 238.76 73.66) (xy 193.04 73.66)
+			(xy 238.76 73.66) (xy 190.5 73.66)
 		)
 		(stroke
@@
 	(polyline
 		(pts
-			(xy 193.04 27.94) (xy 193.04 73.66)
+			(xy 190.5 27.94) (xy 190.5 73.66)
 		)
 		(stroke
@@
 			)
 		)
-		(property "Value" "DMP6023LFG-7"
+		(property "Value" "SQJ457EP-T1_BE3"
 			(at 227.965 40.64 90)
 			(effects
@@
 			)
 		)
-		(property "Footprint" "PCM_EEZ_SMD:TRANS_FDMC8010"
+		(property "Footprint" "PCM_EEZ_SMD:PowerPAK SO-8"
 			(at 211.455 38.1 0)
 			(effects
@@
 			)
 		)
-		(property "DigiKey" "DMP6023LFG-7DICT-ND"
+		(property "DigiKey" "742-SQJ457EP-T1_BE3CT-ND"
 			(at 223.52 38.1 0)
 			(effects
@@
 			)
 		)
-		(property "Mouser" "621-DMP6023LFG-7"
+		(property "Mouser" "78-SQJ457EP-T1_BE3"
 			(at 223.52 38.1 0)
 			(effects
@@
 			)
 		)
-		(property "LCSC" "C526579"
+		(property "LCSC" "C7364386"
 			(at 223.52 38.1 0)
 			(effects
@@
 		(on_board yes)
 		(dnp no)
-		(property "Reference" "C80"
+		(property "Reference" "C79"
 			(at 202.565 96.52 0)
 			(effects
@@
 			(project "EEZ DIB DCP405"
 				(path "/65943c0e-8943-4d2a-93dc-fb4938f73312/55df2794-308a-4204-a97c-7cdafc416b78"
-					(reference "C80")
+					(reference "C79")
 					(unit 1)
 				)
@@
 	(symbol
 		(lib_id "PCM_EEZ_passives:C-EU")
-		(at 203.2 38.1 0)
-		(unit 1)
-		(exclude_from_sim no)
-		(in_bom no)
-		(on_board yes)
-		(dnp yes)
-		(property "Reference" "C79"
-			(at 203.2 38.1 0)
-			(effects
-				(font
-					(size 1.27 1.27)
-				)
-				(justify left bottom)
-			)
-		)
-		(property "Value" "10n"
-			(at 203.2 41.91 0)
-			(effects
-				(font
-					(size 1.27 1.27)
-				)
-				(justify left bottom)
-			)
-		)
-		(property "Footprint" "PCM_EEZ_passives:C_0805_2012Metric"
-			(at 203.2 35.56 0)
-			(effects
-				(font
-					(size 1.27 1.27)
-				)
-				(hide yes)
-			)
-		)
-		(property "Datasheet" ""
-			(at 203.2 35.56 0)
-			(effects
-				(font
-					(size 1.27 1.27)
-				)
-				(hide yes)
-			)
-		)
-		(property "Description" ""
-			(at 203.2 38.1 0)
-			(effects
-				(font
-					(size 1.27 1.27)
-				)
-				(hide yes)
-			)
-		)
-		(property "DigiKey" "490-7194-1-ND "
-			(at 203.2 38.1 0)
-			(effects
-				(font
-					(size 1.27 1.27)
-				)
-				(hide yes)
-			)
-		)
-		(property "Mouser" "710-885012207122"
-			(at 203.2 38.1 0)
-			(effects
-				(font
-					(size 1.27 1.27)
-				)
-				(hide yes)
-			)
-		)
-		(property "TME" "CC0805KRX7R9103"
-			(at 203.2 38.1 0)
-			(effects
-				(font
-					(size 1.27 1.27)
-				)
-				(hide yes)
-			)
-		)
-		(property "LCSC" ""
-			(at 203.2 38.1 0)
-			(effects
-				(font
-					(size 1.27 1.27)
-				)
-				(hide yes)
-			)
-		)
-		(pin "1"
-		)
-		(pin "2"
-		)
-		(instances
-			(project "EEZ DIB DCP405plus"
-				(path "/65943c0e-8943-4d2a-93dc-fb4938f73312/55df2794-308a-4204-a97c-7cdafc416b78"
-					(reference "C79")
-					(unit 1)
-				)
-			)
-		)
-	)
-	(symbol
-		(lib_id "PCM_EEZ_passives:C-EU")
 		(at 198.12 101.6 0)
 		(unit 1)
@@
 		(on_board yes)
 		(dnp no)
-		(property "Reference" "C82"
+		(property "Reference" "C81"
 			(at 223.901 146.939 90)
 			(effects
@@
 			(project "EEZ DIB DCP405"
 				(path "/65943c0e-8943-4d2a-93dc-fb4938f73312/55df2794-308a-4204-a97c-7cdafc416b78"
-					(reference "C82")
+					(reference "C81")
 					(unit 1)
 				)
@@
 	)
 	(symbol
+		(lib_id "PCM_EEZ_discretes:DIODE_ZENER")
+		(at 203.2 40.64 90)
+		(unit 1)
+		(exclude_from_sim no)
+		(in_bom no)
+		(on_board yes)
+		(dnp yes)
+		(property "Reference" "ZD3"
+			(at 201.295 40.64 90)
+			(effects
+				(font
+					(size 1.27 1.27)
+				)
+				(justify left top)
+			)
+		)
+		(property "Value" "BZX384-C15"
+			(at 201.422 42.545 90)
+			(effects
+				(font
+					(size 0.889 0.889)
+				)
+				(justify left top)
+			)
+		)
+		(property "Footprint" "PCM_EEZ_SMD:SOD-323_1P8X1P35_ONS-M"
+			(at 206.375 41.275 0)
+			(effects
+				(font
+					(size 1.27 1.27)
+				)
+				(hide yes)
+			)
+		)
+		(property "Datasheet" ""
+			(at 203.2 40.64 0)
+			(effects
+				(font
+					(size 1.27 1.27)
+				)
+				(hide yes)
+			)
+		)
+		(property "Description" ""
+			(at 203.2 40.64 0)
+			(effects
+				(font
+					(size 1.27 1.27)
+				)
+				(hide yes)
+			)
+		)
+		(property "DigiKey" "1727-4986-1-ND"
+			(at 203.2 40.64 90)
+			(effects
+				(font
+					(size 1.27 1.27)
+				)
+				(hide yes)
+			)
+		)
+		(property "LCSC" "C454989"
+			(at 203.2 40.64 90)
+			(effects
+				(font
+					(size 1.27 1.27)
+				)
+				(hide yes)
+			)
+		)
+		(property "Mouser" "78-BZX384C15-E3-08"
+			(at 203.2 40.64 90)
+			(effects
+				(font
+					(size 1.27 1.27)
+				)
+				(hide yes)
+			)
+		)
+		(property "TME" "BZX384-C15.115"
+			(at 203.2 40.64 90)
+			(effects
+				(font
+					(size 1.27 1.27)
+				)
+				(hide yes)
+			)
+		)
+		(pin "A"
+		)
+		(pin "C"
+		)
+		(instances
+			(project "EEZ DIB DCP405plus"
+				(path "/65943c0e-8943-4d2a-93dc-fb4938f73312/55df2794-308a-4204-a97c-7cdafc416b78"
+					(reference "ZD3")
+					(unit 1)
+				)
+			)
+		)
+	)
+	(symbol
 		(lib_name "R-EU_7")
 		(lib_id "PCM_EEZ_passives:R-EU")
@@
 		(on_board yes)
 		(dnp no)
-		(property "Reference" "C84"
+		(property "Reference" "C83"
 			(at 241.935 99.06 0)
 			(effects
@@
 			(project "EEZ DIB DCP405"
 				(path "/65943c0e-8943-4d2a-93dc-fb4938f73312/55df2794-308a-4204-a97c-7cdafc416b78"
-					(reference "C84")
+					(reference "C83")
 					(unit 1)
 				)
@@
 		(on_board yes)
 		(dnp no)
-		(property "Reference" "C81"
+		(property "Reference" "C80"
 			(at 211.455 95.885 0)
 			(effects
@@
 			(project "EEZ DIB DCP405"
 				(path "/65943c0e-8943-4d2a-93dc-fb4938f73312/55df2794-308a-4204-a97c-7cdafc416b78"
-					(reference "C81")
+					(reference "C80")
 					(unit 1)
 				)
@@
 		(on_board yes)
 		(dnp no)
-		(property "Reference" "C83"
+		(property "Reference" "C82"
 			(at 235.585 98.425 0)
 			(effects
@@
 			(project "EEZ DIB DCP405"
 				(path "/65943c0e-8943-4d2a-93dc-fb4938f73312/55df2794-308a-4204-a97c-7cdafc416b78"
-					(reference "C83")
+					(reference "C82")
 					(unit 1)
 				)
