File: KiCad/Power_pre-regulator.kicad_sch (KiCad schematic)
At the start: 65 parts, among them IC16 LM5145RGYR, Q4 BSC117N08NS5ATMA1, Q5 BSC039N06NSATMA1, Q6 2N7002, Q7 MMBT5401, Q8 SQJ457EP-T1_BE3, X3 B4PS-VH (LF)(SN)

Commit message: #6
Changed lines of the file:
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@@
 	(title_block
 		(title "${project_name}")
-		(date "2026-03-23")
+		(date "2026-03-27")
 		(rev "${project_version}")
 		(company "${project_creator}")
@@
 	(text "100u"
 		(exclude_from_sim no)
-		(at 211.455 103.505 0)
+		(at 211.455 100.965 0)
 		(effects
 			(font
-				(size 1.27 1.27)
+				(size 0.889 0.889)
 				(color 132 0 132 1)
 			)
@@
 		(dnp no)
 		(property "Reference" "C80"
-			(at 211.455 95.885 0)
+			(at 212.725 97.79 0)
 			(effects
 				(font
@@
 		)
 		(property "Value" "EEEFK1J101P"
-			(at 211.455 100.965 0)
+			(at 212.725 99.06 0)
 			(effects
 				(font
@@
 	)
 	(symbol
-		(lib_name "ECAP_1")
 		(lib_id "PCM_EEZ_passives:ECAP")
 		(at 175.26 43.18 90)
@@
 		(dnp no)
 		(property "Reference" "C76"
-			(at 177.8 42.545 90)
+			(at 178.435 42.545 90)
 			(effects
 				(font
@@
 		)
 		(property "Value" "EEEFK1H470P"
-			(at 171.958 46.5074 90)
+			(at 178.435 44.45 90)
 			(effects
 				(font
-					(size 1.27 1.27)
+					(size 0.889 0.889)
 				)
 				(justify right bottom)
@@
 	)
 	(symbol
-		(lib_name "ECAP_2")
 		(lib_id "PCM_EEZ_passives:ECAP")
 		(at 236.22 99.06 0)
@@
 		(dnp no)
 		(property "Reference" "C82"
-			(at 235.585 98.425 0)
+			(at 234.315 100.33 0)
 			(effects
 				(font
@@
 		)
 		(property "Value" "EEEFK1H470P"
-			(at 235.585 103.505 0)
+			(at 234.315 101.6 0)
 			(effects
 				(font

Commit message: OSHWA logo added, KiCad 10 migration
Parts:
- JP7, JP8: value ~ -> (none)

Commit message: #7
Parts:
- R34: now fitted; now in the parts list
Changed lines of the file:
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@@
 	(title_block
 		(title "${project_name}")
-		(date "2026-04-29")
+		(date "2026-04-30")
 		(rev "${project_version}")
 		(company "${project_creator}")
@@
 					(reference "ZD2")
 					(unit 1)
+					(variant
+						(name "Basic")
+						(dnp yes)
+						(in_bom no)
+					)
 				)
 			)
@@
 		(body_style 1)
 		(exclude_from_sim no)
-		(in_bom no)
+		(in_bom yes)
 		(on_board yes)
 		(in_pos_files yes)
-		(dnp yes)
+		(dnp no)
 		(property "Reference" "R34"
 			(at 41.91 29.21 0)
@@
 			)
 		)
+		(property "LCSC" ""
+			(at 43.18 30.48 0)
+			(hide yes)
+			(show_name no)
+			(do_not_autoplace no)
+			(effects
+				(font
+					(size 0.889 0.889)
+				)
+			)
+		)
 		(pin "1"
 		)
@@
 					(reference "R34")
 					(unit 1)
+					(variant
+						(name "Basic")
+						(dnp yes)
+						(in_bom no)
+					)
 				)
 			)

Commit message: BOM and Gerbers update
Parts:
- C76, C82: LCSC (none) -> C278400
- C80: LCSC (none) -> C128460
- D10, D8: LCSC (none) -> C109218
- D9: LCSC (none) -> -
- R40: DigiKey (none) -> YAG1320CT-ND; LCSC (none) -> C859127; Mouser (none) -> 603-RC0805FR-0710RP
Changed lines of the file:
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@@
 			)
 		)
+		(property "DigiKey" "YAG1320CT-ND"
+			(at 170.18 104.14 0)
+			(hide yes)
+			(show_name no)
+			(do_not_autoplace no)
+			(effects
+				(font
+					(size 0.889 0.889)
+				)
+			)
+		)
+		(property "LCSC" "C859127"
+			(at 170.18 104.14 0)
+			(hide yes)
+			(show_name no)
+			(do_not_autoplace no)
+			(effects
+				(font
+					(size 0.889 0.889)
+				)
+			)
+		)
+		(property "Mouser" "603-RC0805FR-0710RP"
+			(at 170.18 104.14 0)
+			(hide yes)
+			(show_name no)
+			(do_not_autoplace no)
+			(effects
+				(font
+					(size 0.889 0.889)
+				)
+			)
+		)
 		(pin "1"
 		)
@@
 			)
 		)
+		(property "LCSC" "C128460"
+			(at 210.82 96.52 0)
+			(hide yes)
+			(show_name no)
+			(do_not_autoplace no)
+			(effects
+				(font
+					(size 0.889 0.889)
+				)
+			)
+		)
 		(pin "+"
 		)
@@
 			)
 		)
+		(property "LCSC" "C109218"
+			(at 223.52 129.54 0)
+			(hide yes)
+			(show_name no)
+			(do_not_autoplace no)
+			(effects
+				(font
+					(size 0.889 0.889)
+				)
+			)
+		)
 		(pin "A"
 		)
@@
 			)
 		)
+		(property "LCSC" "C109218"
+			(at 60.96 73.66 0)
+			(hide yes)
+			(show_name no)
+			(do_not_autoplace no)
+			(effects
+				(font
+					(size 0.889 0.889)
+				)
+			)
+		)
 		(pin "A"
 		)
@@
 			)
 		)
+		(property "LCSC" "-"
+			(at 60.96 81.28 0)
+			(hide yes)
+			(show_name no)
+			(do_not_autoplace no)
+			(effects
+				(font
+					(size 0.889 0.889)
+				)
+			)
+		)
 		(pin "A"
 		)
@@
 			)
 		)
+		(property "LCSC" "C278400"
+			(at 175.26 43.18 90)
+			(hide yes)
+			(show_name no)
+			(do_not_autoplace no)
+			(effects
+				(font
+					(size 0.889 0.889)
+				)
+			)
+		)
 		(pin "+"
 		)
@@
 				)
 			)
+		)
+		(property "LCSC" "C278400"
+			(at 236.22 99.06 0)
+			(hide yes)
+			(show_name no)
+			(do_not_autoplace no)
+			(effects
+				(font
+					(size 0.889 0.889)
+				)
+			)

Commit message: #8, schematics annotated
Parts:
- renumbered Q4 to Q2, Q5 to Q3, Q6 to Q4, Q7 to Q5, Q8 to Q6, R33 to R36, R34 to R37, R35 to R38, R36 to R39, R37 to R40, R38 to R41, R39 to R42, R40 to R43, R41 to R44, R42 to R45, R43 to R46, R44 to R47, R45 to R48, R46 to R49, R47 to R50, R48 to R51, TP9 to TP10, TP10 to TP11, TP11 to TP12, TP12 to TP13, TP8 to TP9
Changed lines of the file:
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@@
 	(title_block
 		(title "${project_name}")
-		(date "2026-05-10")
+		(date "2026-06-26")
 		(rev "${project_version}")
 		(company "${project_creator}")
@@
 		(in_pos_files yes)
 		(dnp yes)
-		(property "Reference" "Q8"
+		(property "Reference" "Q6"
 			(at 223.52 32.258 90)
 			(show_name no)
@@
 			(project "EEZ DIB DCP405plus"
 				(path "/65943c0e-8943-4d2a-93dc-fb4938f73312/55df2794-308a-4204-a97c-7cdafc416b78"
-					(reference "Q8")
+					(reference "Q6")
 					(unit 1)
 				)
@@
 		(in_pos_files yes)
 		(dnp no)
-		(property "Reference" "TP11"
+		(property "Reference" "TP12"
 			(at 222.25 53.34 90)
 			(show_name no)
@@
 			(project "EEZ DIB DCP405plus"
 				(path "/65943c0e-8943-4d2a-93dc-fb4938f73312/55df2794-308a-4204-a97c-7cdafc416b78"
-					(reference "TP11")
+					(reference "TP12")
 					(unit 1)
 				)
@@
 		(in_pos_files yes)
 		(dnp no)
-		(property "Reference" "R38"
+		(property "Reference" "R41"
 			(at 147.32 90.17 90)
 			(show_name no)
@@
 			(project "EEZ DIB DCP405plus"
 				(path "/65943c0e-8943-4d2a-93dc-fb4938f73312/55df2794-308a-4204-a97c-7cdafc416b78"
-					(reference "R38")
+					(reference "R41")
 					(unit 1)
 				)
@@
 		(in_pos_files yes)
 		(dnp no)
-		(property "Reference" "R40"
+		(property "Reference" "R43"
 			(at 171.45 102.235 0)
 			(show_name no)
@@
 			(project "EEZ DIB DCP405plus"
 				(path "/65943c0e-8943-4d2a-93dc-fb4938f73312/55df2794-308a-4204-a97c-7cdafc416b78"
-					(reference "R40")
+					(reference "R43")
 					(unit 1)
 				)
@@
 		(in_pos_files yes)
 		(dnp yes)
-		(property "Reference" "Q6"
+		(property "Reference" "Q4"
 			(at 208.28 52.705 0)
 			(show_name no)
@@
 			(project "EEZ DIB DCP405plus"
 				(path "/65943c0e-8943-4d2a-93dc-fb4938f73312/55df2794-308a-4204-a97c-7cdafc416b78"
-					(reference "Q6")
+					(reference "Q4")
 					(unit 1)
 				)
@@
 		(in_pos_files yes)
 		(dnp no)
-		(property "Reference" "R45"
+		(property "Reference" "R48"
 			(at 226.06 82.55 90)
 			(show_name no)
@@
 			(project "EEZ DIB DCP405plus"
 				(path "/65943c0e-8943-4d2a-93dc-fb4938f73312/55df2794-308a-4204-a97c-7cdafc416b78"
-					(reference "R45")
+					(reference "R48")
 					(unit 1)
 				)
@@
 		(in_pos_files yes)
 		(dnp no)
-		(property "Reference" "R48"
+		(property "Reference" "R51"
 			(at 246.38 135.89 90)
 			(show_name no)
@@
 			(project "EEZ DIB DCP405plus"
 				(path "/65943c0e-8943-4d2a-93dc-fb4938f73312/55df2794-308a-4204-a97c-7cdafc416b78"
-					(reference "R48")
+					(reference "R51")
 					(unit 1)
 				)
@@
 		(in_pos_files yes)
 		(dnp yes)
-		(property "Reference" "R44"
+		(property "Reference" "R47"
 			(at 217.17 63.5 0)
 			(show_name no)
@@
 			(project "EEZ DIB DCP405plus"
 				(path "/65943c0e-8943-4d2a-93dc-fb4938f73312/55df2794-308a-4204-a97c-7cdafc416b78"
-					(reference "R44")
+					(reference "R47")
 					(unit 1)
 				)
@@
 		(in_pos_files yes)
 		(dnp no)
-		(property "Reference" "R46"
+		(property "Reference" "R49"
 			(at 229.87 121.92 0)
 			(show_name no)
@@
 			(project "EEZ DIB DCP405plus"
 				(path "/65943c0e-8943-4d2a-93dc-fb4938f73312/55df2794-308a-4204-a97c-7cdafc416b78"
-					(reference "R46")
+					(reference "R49")
 					(unit 1)
 				)
@@
 		(in_pos_files yes)
 		(dnp no)
-		(property "Reference" "TP10"
+		(property "Reference" "TP11"
 			(at 90.17 22.225 90)
 			(show_name no)
@@
 			(project "EEZ DIB DCP405plus"
 				(path "/65943c0e-8943-4d2a-93dc-fb4938f73312/55df2794-308a-4204-a97c-7cdafc416b78"
-					(reference "TP10")
+					(reference "TP11")
 					(unit 1)
 				)
@@
 		(in_pos_files yes)
 		(dnp no)
-		(property "Reference" "Q5"
+		(property "Reference" "Q3"
 			(at 149.86 101.6 0)
 			(show_name no)
@@
 			(project "EEZ DIB DCP405plus"
 				(path "/65943c0e-8943-4d2a-93dc-fb4938f73312/55df2794-308a-4204-a97c-7cdafc416b78"
-					(reference "Q5")
+					(reference "Q3")
 					(unit 1)
 				)
@@
 		(in_pos_files yes)
 		(dnp no)
-		(property "Reference" "Q7"
+		(property "Reference" "Q5"
 			(at 219.075 135.255 0)
 			(show_name no)
@@
 			(project "EEZ DIB DCP405plus"
 				(path "/65943c0e-8943-4d2a-93dc-fb4938f73312/55df2794-308a-4204-a97c-7cdafc416b78"
-					(reference "Q7")
+					(reference "Q5")
 					(unit 1)
 				)
@@
 		(in_pos_files yes)
 		(dnp no)
-		(property "Reference" "R37"
+		(property "Reference" "R40"
 			(at 93.98 123.19 90)
 			(show_name no)
@@
 			(project "EEZ DIB DCP405plus"
 				(path "/65943c0e-8943-4d2a-93dc-fb4938f73312/55df2794-308a-4204-a97c-7cdafc416b78"
-					(reference "R37")
+					(reference "R40")
 					(unit 1)
 				)
@@
 		(in_pos_files yes)
 		(dnp no)
-		(property "Reference" "TP9"
+		(property "Reference" "TP10"
 			(at 60.325 55.88 0)
 			(show_name no)
@@
 			(project "EEZ DIB DCP405plus"
 				(path "/65943c0e-8943-4d2a-93dc-fb4938f73312/55df2794-308a-4204-a97c-7cdafc416b78"
-					(reference "TP9")
+					(reference "TP10")
 					(unit 1)
 				)
@@
 		(in_pos_files yes)
 		(dnp no)
-		(property "Reference" "#+3V018"
+		(property "Reference" "#+3V020"
 			(at 43.18 68.58 0)
 			(hide yes)
@@
 			(project "EEZ DIB DCP405plus"
 				(path "/65943c0e-8943-4d2a-93dc-fb4938f73312/55df2794-308a-4204-a97c-7cdafc416b78"
-					(reference "#+3V018")
+					(reference "#+3V020")
 					(unit 1)
 				)
@@
 		(in_pos_files yes)
 		(dnp no)
-		(property "Reference" "R34"
+		(property "Reference" "R37"
 			(at 41.91 29.21 0)
 			(show_name no)
@@
 			(project "EEZ DIB DCP405plus"
 				(path "/65943c0e-8943-4d2a-93dc-fb4938f73312/55df2794-308a-4204-a97c-7cdafc416b78"
-					(reference "R34")
+					(reference "R37")
 					(unit 1)
 					(variant
@@
 		(in_pos_files yes)
 		(dnp no)
-		(property "Reference" "R43"
+		(property "Reference" "R46"
 			(at 217.17 121.92 0)
 			(show_name no)
@@
 			(project "EEZ DIB DCP405plus"
 				(path "/65943c0e-8943-4d2a-93dc-fb4938f73312/55df2794-308a-4204-a97c-7cdafc416b78"
-					(reference "R43")
+					(reference "R46")
 					(unit 1)
 				)
@@
 		(in_pos_files yes)
 		(dnp no)
-		(property "Reference" "TP8"
+		(property "Reference" "TP9"
 			(at 60.325 50.8 0)
 			(show_name no)
@@
 			(project "EEZ DIB DCP405plus"
 				(path "/65943c0e-8943-4d2a-93dc-fb4938f73312/55df2794-308a-4204-a97c-7cdafc416b78"
-					(reference "TP8")
+					(reference "TP9")
 					(unit 1)
 				)
@@
 		(in_pos_files yes)
 		(dnp no)
-		(property "Reference" "R39"
+		(property "Reference" "R42"
 			(at 152.4 115.57 90)
 			(show_name no)
@@
 			(project "EEZ DIB DCP405plus"
 				(path "/65943c0e-8943-4d2a-93dc-fb4938f73312/55df2794-308a-4204-a97c-7cdafc416b78"
-					(reference "R39")
+					(reference "R42")
 					(unit 1)
 				)
@@
 		(in_pos_files yes)
 		(dnp no)
-		(property "Reference" "R36"
+		(property "Reference" "R39"
 			(at 69.85 91.44 0)
 			(show_name no)
@@
 			(project "EEZ DIB DCP405plus"
 				(path "/65943c0e-8943-4d2a-93dc-fb4938f73312/55df2794-308a-4204-a97c-7cdafc416b78"
-					(reference "R36")
+					(reference "R39")
 					(unit 1)
 				)
@@
 		(in_pos_files yes)
 		(dnp yes)
-		(property "Reference" "R35"
+		(property "Reference" "R38"
 			(at 53.34 171.45 90)
 			(show_name no)
@@
 			(project "EEZ DIB DCP405plus"
 				(path "/65943c0e-8943-4d2a-93dc-fb4938f73312/55df2794-308a-4204-a97c-7cdafc416b78"
-					(reference "R35")
+					(reference "R38")
 					(unit 1)
 				)
@@
 		(in_pos_files yes)
 		(dnp no)
-		(property "Reference" "Q4"
+		(property "Reference" "Q2"
 			(at 149.86 70.485 0)
 			(show_name no)
@@
 			(project "EEZ DIB DCP405plus"
 				(path "/65943c0e-8943-4d2a-93dc-fb4938f73312/55df2794-308a-4204-a97c-7cdafc416b78"
-					(reference "Q4")
+					(reference "Q2")
 					(unit 1)
 				)
@@
 		(in_pos_files yes)
 		(dnp no)
-		(property "Reference" "R47"
+		(property "Reference" "R50"
 			(at 236.22 135.89 90)
 			(show_name no)
@@
 			(project "EEZ DIB DCP405plus"
 				(path "/65943c0e-8943-4d2a-93dc-fb4938f73312/55df2794-308a-4204-a97c-7cdafc416b78"
-					(reference "R47")
+					(reference "R50")
 					(unit 1)
 				)
@@
 		(in_pos_files yes)
 		(dnp no)
-		(property "Reference" "R41"
+		(property "Reference" "R44"
 			(at 201.93 147.32 0)
 			(show_name no)
@@
 			(project "EEZ DIB DCP405plus"
 				(path "/65943c0e-8943-4d2a-93dc-fb4938f73312/55df2794-308a-4204-a97c-7cdafc416b78"
-					(reference "R41")
+					(reference "R44")
 					(unit 1)
 				)
@@
 		(in_pos_files yes)
 		(dnp yes)
-		(property "Reference" "R33"
+		(property "Reference" "R36"
 			(at 40.64 171.45 90)
 			(show_name no)
@@
 			(project "EEZ DIB DCP405plus"
 				(path "/65943c0e-8943-4d2a-93dc-fb4938f73312/55df2794-308a-4204-a97c-7cdafc416b78"
-					(reference "R33")
+					(reference "R36")
 					(unit 1)
 				)
@@
 		(in_pos_files yes)
 		(dnp yes)
-		(property "Reference" "R42"
+		(property "Reference" "R45"
 			(at 212.09 40.64 0)
 			(show_name no)
@@
 			(project "EEZ DIB DCP405plus"
 				(path "/65943c0e-8943-4d2a-93dc-fb4938f73312/55df2794-308a-4204-a97c-7cdafc416b78"
-					(reference "R42")
+					(reference "R45")
 					(unit 1)
 				)
@@
 		(in_pos_files yes)
 		(dnp no)
-		(property "Reference" "TP12"
+		(property "Reference" "TP13"
 			(at 242.57 85.09 90)
 			(show_name no)
@@
 			(project "EEZ DIB DCP405plus"
 				(path "/65943c0e-8943-4d2a-93dc-fb4938f73312/55df2794-308a-4204-a97c-7cdafc416b78"
-					(reference "TP12")
+					(reference "TP13")
 					(unit 1)
 				)
