File: KiCad/Power_pre-regulator.kicad_sch (KiCad schematic)
At the start: 65 parts, among them IC16 LM5145RGYR, Q2 BSC117N08NS5ATMA1, Q3 BSC039N06NSATMA1, Q4 2N7002, Q5 MMBT5401, Q6 SQJ457EP-T1_BE3, X3 B4PS-VH (LF)(SN)

Commit message: #9
Parts:
- C62, C75: value 470n -> 470n/100V; DigiKey 1276-6482-1-ND -> 587-5014-1-ND; LCSC (none) -> C97926; Mouser 603-CC805KKX7R9BB474 -> 963-HMK212C7474MGHTE; TME CL21B474KBFNNNE -> GRM21BR72A474KA73L
- C74: Mouser 80-C0603C102K5R7040 -> 81-GRT1885C2A102JA2D
- C77, C78, C79: Mouser 810-C3216X7R1HK160AC -> 187-CL32A106KBJNNNE
- R37: value 2R2/2-3W -> 4K7/2W; DigiKey CRM2512-JW-2R2ELFCT-ND -> (none); Mouser 279-35222R2JT -> (none); TME WF25P2R2JTL -> (none); now not fitted; now left out of the parts list
Connections:
- net DC_OUT: now also R36.2; no longer JP7.1
- net POST_OUT+: now also JP7.2; no longer RV1.2
- new net: JP7.1, RV1.2
Other:
- moved on the sheet: JP7, R36, R38, RV1

Commit message: Basic front mask gerbers, two test points, BOM updated
Parts:
- renumbered C61 to C46, C62 to C47, C63 to C48, C64 to C49, C65 to C50, C66 to C51, C67 to C52, C68 to C53, C69 to C54, C70 to C55, C71 to C56, C72 to C57, C73 to C58, C74 to C59, C75 to C60, C76 to C61, C77 to C62, C78 to C63, C79 to C64, C80 to C65, C81 to C66, C82 to C67, C83 to C68, D8 to D4, D9 to D5, D10 to D6, IC16 to IC12, JP9 to JP10, JP7 to JP9, R36 to R26, R37 to R27, R38 to R28, R39 to R29, R40 to R30, R41 to R31, R42 to R32, R43 to R33, R44 to R34, R45 to R35, R46 to R36, R47 to R37, R48 to R38, R49 to R39, R50 to R40, R51 to R41, TP12 to TP10, TP13 to TP11, TP9 to TP7, TP10 to TP8, TP11 to TP9

Commit message: ADC DRDY test point added
Parts:
- renumbered TP9 to TP10, TP10 to TP11, TP11 to TP12, TP7 to TP8, TP8 to TP9
Changed lines of the file:
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@@
 	(title_block
 		(title "${project_name}")
-		(date "2026-09-20")
+		(date "2026-09-21")
 		(rev "${project_version}")
 		(company "${project_creator}")
@@
 		(in_pos_files no)
 		(dnp no)
-		(property "Reference" "TP10"
+		(property "Reference" "TP11"
 			(at 222.25 53.34 90)
 			(show_name no)
@@
 			(project "EEZ DIB DCP405plus"
 				(path "/65943c0e-8943-4d2a-93dc-fb4938f73312/55df2794-308a-4204-a97c-7cdafc416b78"
-					(reference "TP10")
+					(reference "TP11")
 					(unit 1)
 				)
@@
 		(in_pos_files no)
 		(dnp no)
-		(property "Reference" "TP9"
+		(property "Reference" "TP10"
 			(at 90.17 22.225 90)
 			(show_name no)
@@
 			(project "EEZ DIB DCP405plus"
 				(path "/65943c0e-8943-4d2a-93dc-fb4938f73312/55df2794-308a-4204-a97c-7cdafc416b78"
-					(reference "TP9")
+					(reference "TP10")
 					(unit 1)
 				)
@@
 		(in_pos_files no)
 		(dnp no)
-		(property "Reference" "TP8"
+		(property "Reference" "TP9"
 			(at 60.325 55.88 0)
 			(show_name no)
@@
 			(project "EEZ DIB DCP405plus"
 				(path "/65943c0e-8943-4d2a-93dc-fb4938f73312/55df2794-308a-4204-a97c-7cdafc416b78"
-					(reference "TP8")
+					(reference "TP9")
 					(unit 1)
 				)
@@
 		(in_pos_files no)
 		(dnp no)
-		(property "Reference" "TP7"
+		(property "Reference" "TP8"
 			(at 60.325 50.8 0)
 			(show_name no)
@@
 			(project "EEZ DIB DCP405plus"
 				(path "/65943c0e-8943-4d2a-93dc-fb4938f73312/55df2794-308a-4204-a97c-7cdafc416b78"
-					(reference "TP7")
+					(reference "TP8")
 					(unit 1)
 				)
@@
 		(in_pos_files no)
 		(dnp no)
-		(property "Reference" "TP11"
+		(property "Reference" "TP12"
 			(at 242.57 85.09 90)
 			(show_name no)
@@
 			(project "EEZ DIB DCP405plus"
 				(path "/65943c0e-8943-4d2a-93dc-fb4938f73312/55df2794-308a-4204-a97c-7cdafc416b78"
-					(reference "TP11")
+					(reference "TP12")
 					(unit 1)
 				)

Commit message: #10
Parts:
- renumbered TP11 to TP10, TP12 to TP11, TP8 to TP7, TP9 to TP8, TP10 to TP9
Changed lines of the file:
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@@
 	(title_block
 		(title "${project_name}")
-		(date "2026-09-21")
+		(date "2026-10-08")
 		(rev "${project_version}")
 		(company "${project_creator}")
@@
 		(in_pos_files no)
 		(dnp no)
-		(property "Reference" "TP11"
+		(property "Reference" "TP10"
 			(at 222.25 53.34 90)
 			(show_name no)
@@
 			(project "EEZ DIB DCP405plus"
 				(path "/65943c0e-8943-4d2a-93dc-fb4938f73312/55df2794-308a-4204-a97c-7cdafc416b78"
-					(reference "TP11")
+					(reference "TP10")
 					(unit 1)
 				)
@@
 		(in_pos_files no)
 		(dnp no)
-		(property "Reference" "TP10"
+		(property "Reference" "TP9"
 			(at 90.17 22.225 90)
 			(show_name no)
@@
 			(project "EEZ DIB DCP405plus"
 				(path "/65943c0e-8943-4d2a-93dc-fb4938f73312/55df2794-308a-4204-a97c-7cdafc416b78"
-					(reference "TP10")
+					(reference "TP9")
 					(unit 1)
 				)
@@
 		(in_pos_files no)
 		(dnp no)
-		(property "Reference" "TP9"
+		(property "Reference" "TP8"
 			(at 60.325 55.88 0)
 			(show_name no)
@@
 			(project "EEZ DIB DCP405plus"
 				(path "/65943c0e-8943-4d2a-93dc-fb4938f73312/55df2794-308a-4204-a97c-7cdafc416b78"
-					(reference "TP9")
+					(reference "TP8")
 					(unit 1)
 				)
@@
 		(in_pos_files no)
 		(dnp no)
-		(property "Reference" "TP8"
+		(property "Reference" "TP7"
 			(at 60.325 50.8 0)
 			(show_name no)
@@
 			(project "EEZ DIB DCP405plus"
 				(path "/65943c0e-8943-4d2a-93dc-fb4938f73312/55df2794-308a-4204-a97c-7cdafc416b78"
-					(reference "TP8")
+					(reference "TP7")
 					(unit 1)
 				)
@@
 		(in_pos_files no)
 		(dnp no)
-		(property "Reference" "TP12"
+		(property "Reference" "TP11"
 			(at 242.57 85.09 90)
 			(show_name no)
@@
 			(project "EEZ DIB DCP405plus"
 				(path "/65943c0e-8943-4d2a-93dc-fb4938f73312/55df2794-308a-4204-a97c-7cdafc416b78"
-					(reference "TP12")
+					(reference "TP11")
 					(unit 1)
 				)
