File: KiCad/Rsense_protection_power_output.kicad_sch (KiCad schematic)
At the start: 61 parts, among them IC21 SN74LVC2G08DCTR, IC22 LM293D, IC23 OPA376AIDBVR, IC24 SN74LVC1G3157DCKR, IC25 SN74LVC1G3157DCKR, J1 572-0500, J2 572-0100, K1 FTR-C1GA012G-B05 or EE2-12NU-L, Q20 MMBT5551, Q21 MMBT5551, Q22 MMBT5551, Q23 MMBT5401, Q24 2N7002, X4 TBP03R1-350-03BE, X5 ZL263-20DG

Commit message: DIB connector update
Parts:
- J1: footprint PCM_EEZ_connectors:572-0X00 -> PCM_EEZ_connectors:572-0500
- J2: footprint PCM_EEZ_connectors:572-0X00 -> PCM_EEZ_connectors:572-0100
Changed lines of the file:
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@@
 	(title_block
 		(title "${project_name}")
-		(date "2026-01-03")
+		(date "2026-01-06")
 		(rev "${project_version}")
 		(company "${project_creator}")
@@
 			)
 		)
-		(property "Footprint" "PCM_EEZ_connectors:572-0X00"
+		(property "Footprint" "PCM_EEZ_connectors:572-0500"
 			(at 233.68 48.26 0)
 			(effects
@@
 			)
 		)
-		(property "Datasheet" ""
+		(property "Datasheet" "~"
 			(at 233.68 48.26 0)
 			(effects
@@
 			)
 		)
-		(property "Description" ""
+		(property "Description" "Generic connector, single row, 01x02, script generated (kicad-library-utils/schlib/autogen/connector/)"
 			(at 233.68 48.26 0)
 			(effects
@@
 			)
 		)
-		(property "Footprint" "PCM_EEZ_connectors:572-0X00"
+		(property "Footprint" "PCM_EEZ_connectors:572-0100"
 			(at 233.68 76.2 0)
 			(effects
@@
 			)
 		)
-		(property "Description" ""
+		(property "Description" "Generic connector, single row, 01x02, script generated (kicad-library-utils/schlib/autogen/connector/)"
 			(at 233.68 76.2 0)
 			(effects

Commit message: Gerbers update
Parts:
- renumbered C110 to C109, C111 to C110, C112 to C111, C113 to C112, C114 to C113, C115 to C114, C116 to C115, C117 to C116, C118 to C117, C119 to C118, C120 to C119, C121 to C120, C122 to C121, ZD5 to ZD6, ZD6 to ZD7
Changed lines of the file:
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@@
 	(title_block
 		(title "${project_name}")
-		(date "2026-01-06")
+		(date "2026-01-13")
 		(rev "${project_version}")
 		(company "${project_creator}")
@@
 		(on_board yes)
 		(dnp no)
-		(property "Reference" "C113"
+		(property "Reference" "C112"
 			(at 70.739 113.919 90)
 			(effects
@@
 			(project "EEZ DIB DCP405"
 				(path "/65943c0e-8943-4d2a-93dc-fb4938f73312/5ecda23e-3d86-4b9b-8d83-de3653395b33"
-					(reference "C113")
+					(reference "C112")
 					(unit 1)
 				)
@@
 		(on_board yes)
 		(dnp no)
-		(property "Reference" "C116"
+		(property "Reference" "C115"
 			(at 88.519 167.259 90)
 			(effects
@@
 			(project "EEZ DIB DCP405"
 				(path "/65943c0e-8943-4d2a-93dc-fb4938f73312/5ecda23e-3d86-4b9b-8d83-de3653395b33"
-					(reference "C116")
+					(reference "C115")
 					(unit 1)
 				)
@@
 		(on_board yes)
 		(dnp no)
-		(property "Reference" "ZD6"
+		(property "Reference" "ZD7"
 			(at 164.465 60.96 90)
 			(effects
@@
 			(project "EEZ DIB DCP405"
 				(path "/65943c0e-8943-4d2a-93dc-fb4938f73312/5ecda23e-3d86-4b9b-8d83-de3653395b33"
-					(reference "ZD6")
+					(reference "ZD7")
 					(unit 1)
 				)
@@
 		(on_board yes)
 		(dnp no)
-		(property "Reference" "ZD5"
+		(property "Reference" "ZD6"
 			(at 67.945 147.32 90)
 			(effects
@@
 			(project "EEZ DIB DCP405"
 				(path "/65943c0e-8943-4d2a-93dc-fb4938f73312/5ecda23e-3d86-4b9b-8d83-de3653395b33"
-					(reference "ZD5")
+					(reference "ZD6")
 					(unit 1)
 				)
@@
 		(on_board yes)
 		(dnp no)
-		(property "Reference" "C111"
+		(property "Reference" "C110"
 			(at 56.134 119.634 0)
 			(effects
@@
 			(project "EEZ DIB DCP405"
 				(path "/65943c0e-8943-4d2a-93dc-fb4938f73312/5ecda23e-3d86-4b9b-8d83-de3653395b33"
-					(reference "C111")
+					(reference "C110")
 					(unit 1)
 				)
@@
 		(on_board yes)
 		(dnp no)
-		(property "Reference" "C122"
+		(property "Reference" "C121"
 			(at 223.774 69.469 0)
 			(effects
@@
 			(project "EEZ DIB DCP405"
 				(path "/65943c0e-8943-4d2a-93dc-fb4938f73312/5ecda23e-3d86-4b9b-8d83-de3653395b33"
-					(reference "C122")
+					(reference "C121")
 					(unit 1)
 				)
@@
 		(on_board yes)
 		(dnp no)
-		(property "Reference" "C121"
+		(property "Reference" "C120"
 			(at 223.774 56.769 0)
 			(effects
@@
 			(project "EEZ DIB DCP405"
 				(path "/65943c0e-8943-4d2a-93dc-fb4938f73312/5ecda23e-3d86-4b9b-8d83-de3653395b33"
-					(reference "C121")
+					(reference "C120")
 					(unit 1)
 				)
@@
 		(on_board yes)
 		(dnp no)
-		(property "Reference" "C120"
+		(property "Reference" "C119"
 			(at 155.575 52.705 0)
 			(effects
@@
 			(project "EEZ DIB DCP405"
 				(path "/65943c0e-8943-4d2a-93dc-fb4938f73312/5ecda23e-3d86-4b9b-8d83-de3653395b33"
-					(reference "C120")
+					(reference "C119")
 					(unit 1)
 				)
@@
 		(on_board yes)
 		(dnp no)
-		(property "Reference" "C114"
+		(property "Reference" "C113"
 			(at 70.739 129.159 90)
 			(effects
@@
 			(project "EEZ DIB DCP405"
 				(path "/65943c0e-8943-4d2a-93dc-fb4938f73312/5ecda23e-3d86-4b9b-8d83-de3653395b33"
-					(reference "C114")
+					(reference "C113")
 					(unit 1)
 				)
@@
 		(on_board yes)
 		(dnp no)
-		(property "Reference" "C112"
+		(property "Reference" "C111"
 			(at 67.945 40.64 0)
 			(effects
@@
 			(project "EEZ DIB DCP405"
 				(path "/65943c0e-8943-4d2a-93dc-fb4938f73312/5ecda23e-3d86-4b9b-8d83-de3653395b33"
-					(reference "C112")
+					(reference "C111")
 					(unit 1)
 				)
@@
 		(on_board yes)
 		(dnp no)
-		(property "Reference" "C117"
+		(property "Reference" "C116"
 			(at 109.855 86.36 0)
 			(effects
@@
 			(project "EEZ DIB DCP405"
 				(path "/65943c0e-8943-4d2a-93dc-fb4938f73312/5ecda23e-3d86-4b9b-8d83-de3653395b33"
-					(reference "C117")
+					(reference "C116")
 					(unit 1)
 				)
@@
 		(on_board yes)
 		(dnp no)
-		(property "Reference" "C118"
+		(property "Reference" "C117"
 			(at 117.475 33.02 0)
 			(effects
@@
 			(project "EEZ DIB DCP405"
 				(path "/65943c0e-8943-4d2a-93dc-fb4938f73312/5ecda23e-3d86-4b9b-8d83-de3653395b33"
-					(reference "C118")
+					(reference "C117")
 					(unit 1)
 				)
@@
 		(on_board yes)
 		(dnp no)
-		(property "Reference" "C115"
+		(property "Reference" "C114"
 			(at 88.519 129.159 90)
 			(effects
@@
 			(project "EEZ DIB DCP405"
 				(path "/65943c0e-8943-4d2a-93dc-fb4938f73312/5ecda23e-3d86-4b9b-8d83-de3653395b33"
-					(reference "C115")
+					(reference "C114")
 					(unit 1)
 				)
@@
 		(on_board yes)
 		(dnp no)
-		(property "Reference" "C110"
+		(property "Reference" "C109"
 			(at 38.354 119.634 0)
 			(effects
@@
 			(project "EEZ DIB DCP405"
 				(path "/65943c0e-8943-4d2a-93dc-fb4938f73312/5ecda23e-3d86-4b9b-8d83-de3653395b33"
-					(reference "C110")
+					(reference "C109")
 					(unit 1)
 				)
@@
 		(on_board yes)
 		(dnp no)
-		(property "Reference" "C119"
+		(property "Reference" "C118"
 			(at 149.225 64.77 0)
 			(effects
@@
 			(project "EEZ DIB DCP405"
 				(path "/65943c0e-8943-4d2a-93dc-fb4938f73312/5ecda23e-3d86-4b9b-8d83-de3653395b33"
-					(reference "C119")
+					(reference "C118")
 					(unit 1)
 				)

Commit message: #2, #3, image of the assembled module
Parts:
- added R144: 220R, PCM_EEZ_passives:R_0805_2012Metric, symbol PCM_EEZ_passives:R-EU
- R119: value 470R -> 330R
- R121: value 1K2 -> 1K
Connections:
- net GND: now also R144.1
- net at LED2.GC, LED2.RC, R119.2: now also R144.2
Other:
- moved on the sheet: R119
Changed lines of the file:
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@@
 	(title_block
 		(title "${project_name}")
-		(date "2026-02-25")
+		(date "2026-03-01")
 		(rev "${project_version}")
 		(company "${project_creator}")
@@
 	)
 	(junction
-		(at 187.96 132.08)
-		(diameter 0)
-		(color 0 0 0 0)
-	)
-	(junction
 		(at 177.8 71.12)
 		(diameter 0)
@@
 	)
 	(junction
+		(at 187.96 134.62)
+		(diameter 0)
+		(color 0 0 0 0)
+	)
+	(junction
 		(at 45.72 157.48)
 		(diameter 0)
@@
 	)
 	(junction
+		(at 208.28 134.62)
+		(diameter 0)
+		(color 0 0 0 0)
+	)
+	(junction
 		(at 180.34 50.8)
 		(diameter 0)
@@
 	)
 	(junction
+		(at 187.96 129.54)
+		(diameter 0)
+		(color 0 0 0 0)
+	)
+	(junction
 		(at 101.6 149.86)
 		(diameter 0)
@@
 	(wire
 		(pts
+			(xy 187.96 134.62) (xy 187.96 137.16)
+		)
+		(stroke
+			(width 0)
+			(type default)
+		)
+	)
+	(wire
+		(pts
 			(xy 142.24 83.82) (xy 172.72 83.82)
 		)
@@
 	(wire
 		(pts
+			(xy 187.96 134.62) (xy 195.58 134.62)
+		)
+		(stroke
+			(width 0)
+			(type default)
+		)
+	)
+	(wire
+		(pts
 			(xy 144.78 88.9) (xy 144.78 93.98)
 		)
@@
 	(wire
 		(pts
-			(xy 190.5 132.08) (xy 187.96 132.08)
+			(xy 190.5 129.54) (xy 187.96 129.54)
 		)
 		(stroke
@@
 	(wire
 		(pts
-			(xy 200.66 132.08) (xy 203.2 132.08)
+			(xy 200.66 129.54) (xy 208.28 129.54)
 		)
 		(stroke
@@
 	(wire
 		(pts
-			(xy 203.2 132.08) (xy 203.2 134.62)
+			(xy 208.28 129.54) (xy 208.28 134.62)
 		)
 		(stroke
@@
 	(wire
 		(pts
-			(xy 187.96 132.08) (xy 187.96 137.16)
+			(xy 187.96 129.54) (xy 187.96 134.62)
 		)
 		(stroke
@@
 	(wire
 		(pts
-			(xy 187.96 127) (xy 187.96 132.08)
+			(xy 187.96 127) (xy 187.96 129.54)
 		)
 		(stroke
@@
 	(wire
 		(pts
+			(xy 205.74 134.62) (xy 208.28 134.62)
+		)
+		(stroke
+			(width 0)
+			(type default)
+		)
+	)
+	(wire
+		(pts
 			(xy 142.24 88.9) (xy 144.78 88.9)
 		)
@@
 			)
 		)
-		(property "Value" "1K2"
+		(property "Value" "1K"
 			(at 255.27 130.81 0)
 			(effects
@@
 	)
 	(symbol
+		(lib_id "PCM_EEZ_passives:R-EU")
+		(at 200.66 134.62 90)
+		(mirror x)
+		(unit 1)
+		(exclude_from_sim no)
+		(in_bom yes)
+		(on_board yes)
+		(dnp no)
+		(property "Reference" "R144"
+			(at 200.66 133.35 90)
+			(effects
+				(font
+					(size 1.27 1.27)
+				)
+				(justify bottom)
+			)
+		)
+		(property "Value" "220R"
+			(at 200.66 135.89 90)
+			(effects
+				(font
+					(size 1.27 1.27)
+				)
+				(justify top)
+			)
+		)
+		(property "Footprint" "PCM_EEZ_passives:R_0805_2012Metric"
+			(at 200.66 134.62 0)
+			(effects
+				(font
+					(size 1.27 1.27)
+				)
+				(hide yes)
+			)
+		)
+		(property "Datasheet" ""
+			(at 200.66 134.62 0)
+			(effects
+				(font
+					(size 1.27 1.27)
+				)
+				(hide yes)
+			)
+		)
+		(property "Description" ""
+			(at 200.66 134.62 0)
+			(effects
+				(font
+					(size 1.27 1.27)
+				)
+				(hide yes)
+			)
+		)
+		(property "DigiKey" "311-470CRCT-ND"
+			(at 200.66 134.62 0)
+			(effects
+				(font
+					(size 1.27 1.27)
+				)
+				(hide yes)
+			)
+		)
+		(property "Mouser" "71-CRCW0805470RFKEB"
+			(at 200.66 134.62 0)
+			(effects
+				(font
+					(size 1.27 1.27)
+				)
+				(hide yes)
+			)
+		)
+		(property "TME" "RC0805FR-07470R"
+			(at 200.66 134.62 0)
+			(effects
+				(font
+					(size 1.27 1.27)
+				)
+				(hide yes)
+			)
+		)
+		(pin "1"
+		)
+		(pin "2"
+		)
+		(instances
+			(project "EEZ DIB DCP405plus"
+				(path "/65943c0e-8943-4d2a-93dc-fb4938f73312/5ecda23e-3d86-4b9b-8d83-de3653395b33"
+					(reference "R144")
+					(unit 1)
+				)
+			)
+		)
+	)
+	(symbol
 		(lib_id "PCM_EEZ_TI:OPA376AIDBVR")
 		(at 91.44 149.86 0)
@@
 	(symbol
 		(lib_id "PCM_EEZ_symbols:GND")
-		(at 203.2 137.16 0)
-		(mirror y)
+		(at 208.28 137.16 0)
 		(unit 1)
 		(exclude_from_sim no)
@@
 		(dnp no)
 		(property "Reference" "#SUPPLY066"
-			(at 203.2 137.16 0)
+			(at 208.28 137.16 0)
 			(effects
 				(font
@@
 		)
 		(property "Value" "GND"
-			(at 201.295 138.43 0)
+			(at 210.185 138.43 0)
 			(effects
 				(font
@@
 		)
 		(property "Footprint" ""
-			(at 203.2 137.16 0)
+			(at 208.28 137.16 0)
 			(effects
 				(font
@@
 		)
 		(property "Datasheet" ""
-			(at 203.2 137.16 0)
+			(at 208.28 137.16 0)
 			(effects
 				(font
@@
 		)
 		(property "Description" ""
-			(at 203.2 137.16 0)
+			(at 208.28 137.16 0)
 			(effects
 				(font
@@
 	(symbol
 		(lib_id "PCM_EEZ_passives:R-EU")
-		(at 195.58 132.08 90)
+		(at 195.58 129.54 90)
 		(mirror x)
 		(unit 1)
@@
 		(dnp no)
 		(property "Reference" "R119"
-			(at 195.58 130.81 90)
+			(at 195.58 128.27 90)
 			(effects
 				(font
@@
 			)
 		)
-		(property "Value" "470R"
-			(at 195.58 133.35 90)
+		(property "Value" "330R"
+			(at 195.58 130.81 90)
 			(effects
 				(font
@@
 		)
 		(property "Footprint" "PCM_EEZ_passives:R_0805_2012Metric"
-			(at 195.58 132.08 0)
+			(at 195.58 129.54 0)
 			(effects
 				(font
@@
 		)
 		(property "Datasheet" ""
-			(at 195.58 132.08 0)
+			(at 195.58 129.54 0)
 			(effects
 				(font
@@
 		)
 		(property "Description" ""
-			(at 195.58 132.08 0)
+			(at 195.58 129.54 0)
 			(effects
 				(font
@@
 		)
 		(property "DigiKey" "311-470CRCT-ND"
-			(at 195.58 132.08 0)
+			(at 195.58 129.54 0)
 			(effects
 				(font
@@
 		)
 		(property "Mouser" "71-CRCW0805470RFKEB"
-			(at 195.58 132.08 0)
+			(at 195.58 129.54 0)
 			(effects
 				(font
@@
 		)
 		(property "TME" "RC0805FR-07470R"
-			(at 195.58 132.08 0)
+			(at 195.58 129.54 0)
 			(effects
 				(font
