File: KiCad/Rsense_protection_power_output.kicad_sch (KiCad schematic)
At the start: 66 parts, among them IC21 SN74LVC2G08DCTR, IC22 LM293D, IC23 OPA376AIDBVR, IC24 SN74LVC1G3157DCKR, IC25 SN74LVC1G3157DCKR, J1 572-0500, J2 572-0100, K1 FTR-C1GA012G-B05 or EE2-12NU-L, Q18 MMBT5551, Q19 MMBT5551, Q20 MMBT5551, Q21 MMBT5401, Q22 2N7002, X4 TBP03R1-350-03BE, X5 ZL263-20DG

Commit message: #9
Parts:
- C118: value 470n -> 470n/100V; DigiKey 1276-6482-1-ND -> 587-5014-1-ND; LCSC (none) -> C97926; Mouser 603-CC805KKX7R9BB474 -> 963-HMK212C7474MGHTE; TME CL21B474KBFNNNE -> GRM21BR72A474KA73L

Commit message: Basic front mask gerbers, two test points, BOM updated
Parts:
- renumbered C115 to C100, C116 to C101, C117 to C102, C118 to C103, C119 to C104, C120 to C105, C121 to C106, C109 to C94, C110 to C95, C111 to C96, C112 to C97, C113 to C98, C114 to C99, D20 to D16, D21 to D17, IC21 to IC17, IC22 to IC18, IC23 to IC19, IC24 to IC20, IC25 to IC21, JP10 to JP11, JP11 to JP12, R110 to R100, R111 to R101, R112 to R102, R113 to R103, R114 to R104, R115 to R105, R116 to R106, R117 to R107, R118 to R108, R119 to R109, R120 to R110, R121 to R111, R122 to R112, R123 to R113, R124 to R114, R125 to R115, R126 to R116, R127 to R117, R128 to R118, R129 to R119, R102 to R92, R103 to R93, R104 to R94, R105 to R95, R106 to R96, R107 to R97, R108 to R98, R109 to R99, TP14 to TP12, TP15 to TP13

Commit message: ADC DRDY test point added
Parts:
- renumbered TP12 to TP13, TP13 to TP14
Changed lines of the file:
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@@
 	(title_block
 		(title "${project_name}")
-		(date "2026-09-20")
+		(date "2026-09-21")
 		(rev "${project_version}")
 		(company "${project_creator}")
@@
 		(in_pos_files no)
 		(dnp no)
-		(property "Reference" "TP12"
+		(property "Reference" "TP13"
 			(at 41.91 137.795 90)
 			(show_name no)
@@
 			(project "EEZ DIB DCP405plus"
 				(path "/65943c0e-8943-4d2a-93dc-fb4938f73312/5ecda23e-3d86-4b9b-8d83-de3653395b33"
-					(reference "TP12")
+					(reference "TP13")
 					(unit 1)
 				)
@@
 		(in_pos_files no)
 		(dnp no)
-		(property "Reference" "TP13"
+		(property "Reference" "TP14"
 			(at 46.99 151.765 90)
 			(show_name no)
@@
 			(project "EEZ DIB DCP405plus"
 				(path "/65943c0e-8943-4d2a-93dc-fb4938f73312/5ecda23e-3d86-4b9b-8d83-de3653395b33"
-					(reference "TP13")
+					(reference "TP14")
 					(unit 1)
 				)

Commit message: #10
Parts:
- renumbered TP13 to TP12, TP14 to TP13
Changed lines of the file:
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@@
 	(title_block
 		(title "${project_name}")
-		(date "2026-09-21")
+		(date "2026-10-08")
 		(rev "${project_version}")
 		(company "${project_creator}")
@@
 		(in_pos_files no)
 		(dnp no)
-		(property "Reference" "TP13"
+		(property "Reference" "TP12"
 			(at 41.91 137.795 90)
 			(show_name no)
@@
 			(project "EEZ DIB DCP405plus"
 				(path "/65943c0e-8943-4d2a-93dc-fb4938f73312/5ecda23e-3d86-4b9b-8d83-de3653395b33"
-					(reference "TP13")
+					(reference "TP12")
 					(unit 1)
 				)
@@
 		(in_pos_files no)
 		(dnp no)
-		(property "Reference" "TP14"
+		(property "Reference" "TP13"
 			(at 46.99 151.765 90)
 			(show_name no)
@@
 			(project "EEZ DIB DCP405plus"
 				(path "/65943c0e-8943-4d2a-93dc-fb4938f73312/5ecda23e-3d86-4b9b-8d83-de3653395b33"
-					(reference "TP14")
+					(reference "TP13")
 					(unit 1)
 				)
